File: 60B/60B.kicad_sch (KiCad schematic)
At the start: 150 parts

Commit message: working on tako i3
Parts:
- added D76, D77, D78: LED, LED_THT:LED_D3.0mm, symbol Device:LED
- added H1, H2, H3, H4: MountingHole_Pad, MountingHole:MountingHole_2.2mm_M2_Pad, symbol Mechanical:MountingHole_Pad
- added RV1: R_Potentiometer_MountingPin, Potentiometer_THT:Potentiometer_Bourns_PTA4543_Single_Slide, symbol Device:R_Potentiometer_MountingPin
- added S14, S43, S46, S47, S65, S66, S69, S70: MX_stab, PCM_marbastlib-mx:STAB_MX_P_2u, symbol marbastlib-mx:MX_stab
- added U1: Bonsai-C4-extended, shoonies_parts:Bonsai_C4_extended_THT, symbol Bonsai_C4:Bonsai-C4-extended
- D43, D45: now not fitted; now left out of the parts list
- D44, D46: now fitted; now in the parts list
Connections:
- net ROW4: now reaches D61.1 (K), D62.1 (K), D63.1 (K), D64.1 (K), D65.1 (K), D66.1 (K), D67.1 (K), D68.1 (K), D69.1 (K), D70.1 (K), D71.1 (K), D72.1 (K), D73.1 (K), D74.1 (K), D75.1 (K)
- net ROW4: now also U1.1 (B7_PD3)
- net COL5: now reaches MX21.2, MX36.2, MX52.2, MX6.2, MX67.2
- net COL5: now also U1.24 (A1)
- net ROW1: now reaches D16.1 (K), D17.1 (K), D18.1 (K), D19.1 (K), D20.1 (K), D21.1 (K), D22.1 (K), D23.1 (K), D24.1 (K), D25.1 (K), D26.1 (K), D27.1 (K), D28.1 (K), D29.1 (K)
- net ROW1: now also U1.6 (B6_PD0)
- net at D45.2 (A), D46.2 (A), MX46.1: now also MX45.2; no longer MX45.1
- net COL13: now reaches MX14.2, MX15.2, MX29.2, MX46.2, MX60.2, MX75.2
- net COL13: now also MX45.1, U1.39 (A13); no longer MX45.2
- net COL9: now reaches MX10.2, MX25.2, MX40.2, MX56.2, MX71.2
- net COL9: now also U1.35 (C14)
- net ROW2: now reaches D46.1 (K)
- net ROW2: now also D30.1 (K), D31.1 (K), D32.1 (K), D33.1 (K), D34.1 (K), D35.1 (K), D36.1 (K), D37.1 (K), D38.1 (K), D39.1 (K), D40.1 (K), D41.1 (K), D42.1 (K), D43.1 (K), D44.1 (K), D45.1 (K), U1.5 (B9_PD1)
- net ROW3: now reaches D47.1 (K), D48.1 (K), D49.1 (K), D50.1 (K), D51.1 (K), D52.1 (K), D53.1 (K), D54.1 (K), D55.1 (K), D56.1 (K), D57.1 (K), D58.1 (K), D59.1 (K), D60.1 (K)
- net ROW3: now also U1.2 (A15_PD2)
- net COL8: now reaches MX24.2, MX39.2, MX55.2, MX69.2, MX70.2, MX9.2
- net COL8: now also U1.28 (B1)
- net COL0: now reaches MX1.2, MX16.2, MX30.2, MX47.2, MX61.2
- net COL0: now also MX31.2, U1.12 (B0)
- net COL1: now reaches MX17.2, MX2.2, MX32.2, MX48.2, MX62.2
- net COL1: now also U1.21 (A7)
- net COL7: now reaches MX23.2, MX38.2, MX54.2, MX8.2
- net COL7: now also U1.27 (B15)
- net COL10: now reaches MX11.2, MX26.2, MX41.2, MX57.2, MX72.2
- net COL10: now also U1.36 (C15)
- net ROW0: now reaches D1.1 (K), D10.1 (K), D11.1 (K), D12.1 (K), D13.1 (K), D14.1 (K), D2.1 (K), D3.1 (K), D4.1 (K), D5.1 (K), D6.1 (K), D7.1 (K), D8.1 (K), D9.1 (K)
- net ROW0: now also U1.7 (A4)
- net COL2: now reaches MX18.2, MX3.2, MX33.2, MX49.2, MX63.2
- net COL2: now also U1.25 (B13)
- net COL6: now reaches MX22.2, MX37.2, MX53.2, MX68.2, MX7.2
- net COL6: now also U1.26 (B14)
- net COL12: now reaches MX13.2, MX28.2, MX43.2, MX44.2, MX59.2, MX74.2
- net COL12: now also U1.38 (A14)
- net at D31.2 (A), MX31.1: now also D30.2 (A), MX30.1
- net COL4: now reaches MX20.2, MX35.2, MX5.2, MX51.2, MX65.2, MX66.2
- net COL4: now also U1.22 (A6)
- net COL11: now reaches MX12.2, MX27.2, MX42.2, MX58.2, MX73.2
- net COL11: now also U1.37 (A2)
- net COL3: now reaches MX19.2, MX34.2, MX4.2, MX50.2, MX64.2
- net COL3: now also U1.23 (A5)
- new net +3.3V: RV1.3, U1.20 (+3.3V)
- new net GND: D76.1 (K), D77.1 (K), D78.1 (K), H1.1, H2.1, H3.1, H4.1, RV1.1, RV1.MP (MountPin), U1.18 (GND), U1.3 (GND), U1.4 (GND)
- new net LED1: D76.2 (A), U1.30 (B3_SCK)
- new net LED2: D77.2 (A), U1.31 (B4_MISO)
- new net LED3: D78.2 (A), U1.32 (B5_MOSI)
- new net POT: RV1.2, U1.29 (A0_FRAM_CS)
Other:
- moved on the sheet: D1, D10, D11, D12, D13, D14, D15, D16, D17, D18, D19, D2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
