File: template/i7_uni/i7_uni.kicad_sch (KiCad schematic)
At the start: 31 parts, among them J1 Conn_JST, J2 Conn_DEBUG, SW1 MX_SW, U1 RP2040, U2 XC6206PxxxMR, U3 SRV05-4, U4 W25Q128JVS, Y1 Crystal_GND24

Commit message: i7_uni pause
Parts:
- removed U3: SRV05-4, PCM_marbastlib-various:SOT-23-6-routable, symbol PCM_marbastlib-various:SRV05-4
- added C10, C2, C8, C9: 100n, Capacitor_SMD:C_0402_1005Metric, symbol Device:C_Small
- added D2, D3, D4: D, Diode_SMD:D_SOD-123, symbol Device:D_Small
- added S2, S3, S4: MX_S, PCM_marbastlib-mx:STAB_MX_P_2u, symbol PCM_marbastlib-mx:MX_stab
- added SW2, SW3, SW4: MX_SW, PCM_marbastlib-mx:SW_MX_HS_S_CPG151101S11_1u, symbol PCM_marbastlib-mx:MX_SW_solder
- C1: renamed from C4; footprint (none) -> Capacitor_SMD:C_0402_1005Metric
- C11: renamed from C9; footprint (none) -> Capacitor_SMD:C_0402_1005Metric
- C12: renamed from C1; footprint (none) -> Capacitor_SMD:C_0402_1005Metric
- C13: renamed from C2; footprint (none) -> Capacitor_SMD:C_0402_1005Metric
- C14: renamed from C12; footprint (none) -> Capacitor_SMD:C_0402_1005Metric
- C15: renamed from C10; footprint (none) -> Capacitor_SMD:C_0402_1005Metric
- C16: renamed from C11; footprint (none) -> Capacitor_SMD:C_0402_1005Metric
- C3: renamed from C5; footprint (none) -> Capacitor_SMD:C_0402_1005Metric
- C4: renamed from C3; footprint (none) -> Capacitor_SMD:C_0603_1608Metric
- C5: renamed from C6; footprint (none) -> Capacitor_SMD:C_0402_1005Metric
- C6: renamed from C7; footprint (none) -> Capacitor_SMD:C_0402_1005Metric
- C7: renamed from C8; footprint (none) -> Capacitor_SMD:C_0402_1005Metric
- D1: footprint (none) -> Diode_SMD:D_SOD-123
- J1: value Conn_JST -> ZX-SH1.0-4PWT; footprint (none) -> Connector_JST:JST_SH_SM04B-SRSS-TB_1x04-1MP_P1.00mm_Horizontal
- J2: footprint (none) -> Connector_PinHeader_1.00mm:PinHeader_1x05_P1.00mm_Vertical; now not fitted; now left out of the parts list
- PSW1: value PSW_RST -> SKRPACE010; footprint (none) -> Button_Switch_SMD:SW_Push_1P1T_NO_Vertical_Wuerth_434133025816
- PSW2: value PSW_BOOT -> SKRPACE010; footprint (none) -> Button_Switch_SMD:SW_Push_1P1T_NO_Vertical_Wuerth_434133025816
- R1: renamed from R2; footprint (none) -> Resistor_SMD:R_0402_1005Metric
- R2: renamed from R3; footprint (none) -> Resistor_SMD:R_0402_1005Metric
- R3: renamed from R1; footprint (none) -> Resistor_SMD:R_0402_1005Metric
- R4, R6: footprint (none) -> Resistor_SMD:R_0402_1005Metric
- R5: renamed from R7; footprint (none) -> Resistor_SMD:R_0402_1005Metric
- R7: renamed from R5; footprint (none) -> Resistor_SMD:R_0402_1005Metric
- S1: footprint PCM_marbastlib-mx:STAB_MX_P_6.25u -> PCM_marbastlib-mx:STAB_MX_P_2u; now not fitted; now left out of the parts list
- SW1: footprint PCM_marbastlib-mx:SW_MX_1u -> PCM_marbastlib-mx:SW_MX_HS_S_CPG151101S11_1u
- U1: renamed from U2; value XC6206PxxxMR -> XC6206P332MR-G
- Y1: footprint (none) -> Crystal:Crystal_SMD_3225-4Pin_3.2x2.5mm
- renumbered U1 to U2, U4 to U3
Connections:
- net +1V1: now also C2.1
- net +3V3: now also C10.1, C8.1, C9.1
- net GND: now also C10.2, C2.2, C8.2, C9.2
- net at D1.2 (A): now also SW1.1; no longer SW1.2
- new net: D2.2 (A), SW2.1
- new net: D3.2 (A), SW3.1
- new net: D4.2 (A), SW4.1
- no-connect marks 2 -> 0
Other:
- moved on the sheet: C1, C11, C12, C13, C14, C15, C16, C3, C4, C5, C6, C7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
