File: template/i8/i8.kicad_sch (KiCad schematic)
At the start: 43 parts, among them J1 ZX-SH1.0-4PWT, J2 Conn_DEBUG, SW1 MX_SW, SW2 MX_SW, SW3 MX_SW, SW4 MX_SW, U1 RP2040, U2 XC6206P332MR-G, U3 W25Q128JVS, Y1 Crystal_GND24

Commit message: i8 development
Parts:
- J2: footprint Connector_PinHeader_1.00mm:PinHeader_1x05_P1.00mm_Vertical -> Connector_PinHeader_1.27mm:PinHeader_1x05_P1.27mm_Vertical
Connections:
- net GND: now also J2.1 (Pin_1); no longer J2.3 (Pin_3)
- net RST: now also J2.5 (Pin_5); no longer J2.1 (Pin_1)
- net SWC: now also J2.3 (Pin_3); no longer J2.4 (Pin_4)
- net SWD: now also J2.4 (Pin_4); no longer J2.5 (Pin_5)
Other:
- moved on the sheet: C1, C10, C11, C12, C13, C14, C15, C16, C2, C3, C4, C5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
