File: template/i8/_autosave-i8.kicad_sch (KiCad schematic)
At the start: 44 parts, among them J1 ZX-SH1.0-4PWT, J2 Conn_DEBUG, SW1 MX_SW, SW2 MX_SW, SW3 MX_SW, SW4 MX_SW, U1 XC6206P332MR-G, U2 RP2040, U3 W25Q16JVUXIQ, Y1 Crystal_GND24

Commit message: downgraded flash chip
Parts:
- PSW1: value SKRPACE010 -> REST; footprint Button_Switch_SMD:SW_Push_1P1T_NO_Vertical_Wuerth_434133025816 -> Connector_PinHeader_1.27mm:PinHeader_1x02_P1.27mm_Vertical
- PSW2: value SKRPACE010 -> BOOT; footprint Button_Switch_SMD:SW_Push_1P1T_NO_Vertical_Wuerth_434133025816 -> Connector_PinHeader_1.27mm:PinHeader_1x02_P1.27mm_Vertical
Changed lines of the file:
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@@
 			)
 		)
-		(property "Value" "SKRPACE010"
+		(property "Value" "BOOT"
 			(at 254 245.5488 0)
 			(effects
@@
 			)
 		)
-		(property "Footprint" "Button_Switch_SMD:SW_Push_1P1T_NO_Vertical_Wuerth_434133025816"
+		(property "Footprint" "Connector_PinHeader_1.27mm:PinHeader_1x02_P1.27mm_Vertical"
 			(at 254 245.11 0)
 			(effects
@@
 			)
 		)
-		(property "Value" "SKRPACE010"
+		(property "Value" "REST"
 			(at 260.35 222.6888 0)
 			(effects
@@
 			)
 		)
-		(property "Footprint" "Button_Switch_SMD:SW_Push_1P1T_NO_Vertical_Wuerth_434133025816"
+		(property "Footprint" "Connector_PinHeader_1.27mm:PinHeader_1x02_P1.27mm_Vertical"
 			(at 260.35 222.25 0)
 			(effects
