File: template/i8/i8.kicad_pcb (KiCad board)
At the start: 2 copper layers, 50 x 50 mm, 28 parts, among them J1 ZX-SH1.0-4PWT, SW1 MX_SW, U1 XC6206P332MR-G, U2 RP2040, U3 W25Q16JVUXIQ, Y1 Crystal_GND24

Commit message: prying voltage regulator
Parts:
- added J2: Conn_DEBUG, Connector_PinHeader_1.27mm:PinHeader_1x05_P1.27mm_Vertical, F.Cu at (5.08, 6.20)
- added PSW1: REST, Connector_PinHeader_1.27mm:PinHeader_1x02_P1.27mm_Vertical, F.Cu at (-19.4, -0.20)
- added PSW2: BOOT, Connector_PinHeader_1.27mm:PinHeader_1x02_P1.27mm_Vertical, F.Cu at (-17.8, -0.20)
- added R3: 5.1k, Resistor_SMD:R_0402_1005Metric, F.Cu at (-38.4, 0.41)
- added R5: 5.1k, Resistor_SMD:R_0402_1005Metric, F.Cu at (-38.4, 2.40)
- added R6: 5.1k, Resistor_SMD:R_0402_1005Metric, F.Cu at (-38.4, 4.39)
- added R7: 1k, Resistor_SMD:R_0402_1005Metric, F.Cu at (-38.4, 6.38)
- D1, S1, SW1: moved to F.Cu
- moved S1 182.0 mm to (-60.9, -18.8), turned to 0 degrees
- moved D1 165.0 mm to (-52.3, -1.75), turned to 0 degrees
- moved SW1 152.9 mm to (-67.4, -0.55), turned to 0 degrees
- moved U1 7.13 mm to (-11.3, -9.47), turned to 135 degrees
- moved C13 5.25 mm to (-13.6, -8.75), turned to -45 degrees
- moved C14 3.79 mm to (-12.0, -7.13), turned to 135 degrees
- moved C10 0.71 mm to (-5.58, 1.91)
- moved C17 0.71 mm to (8.44, 4.71)
- moved C2 0.71 mm to (2.77, 4.72)
- moved C8 0.71 mm to (3.42, 4.07)
- moved J1 0.71 mm to (-14.1, -14.1)
- moved R4 0.71 mm to (5.10, 4.43)
- moved C9 0.71 mm to (-3.04, 4.45)
- moved Y1 0.71 mm to (6.63, 2.90)
- moved C16 0.71 mm to (8.16, 1.37)
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Routing:
- net +3V3: track 23.4 -> 57.2 mm, vias 0 -> 1
- net GND: track 22.8 -> 29.1 mm, vias 21 -> 20
- net +5V: track 10.7 -> 4.64 mm
- net SWC: track 0.89 -> 5.08 mm
- net RST: track 0.67 -> 4.28 mm
- net SWD: track 0.67 -> 3.16 mm, vias 1 -> 0
- net GPIO22: track 0.70 -> 0.00 mm, vias 1 -> 0
- net GPIO21: track 0.70 -> 0.00 mm, vias 1 -> 0
- net GPIO29_ADC3: track 0.70 -> 0.00 mm, vias 1 -> 0
- net GPIO7: track 0.68 -> 0.00 mm, vias 1 -> 0
- net GPIO0: track 0.68 -> 0.00 mm, vias 1 -> 0
- net GPIO8: track 0.67 -> 0.00 mm, vias 1 -> 0
- net GPIO15: track 0.67 -> 0.00 mm, vias 1 -> 0
- net GPIO14: track 0.67 -> 0.00 mm, vias 1 -> 0
- net GPIO16: track 0.67 -> 0.00 mm, vias 1 -> 0
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
Commit message: i8 development
Parts:
- removed D1: 1N4148W, Diode_SMD:D_SOD-123
- removed S1: MX_S, PCM_marbastlib-mx:STAB_MX_P_2u
- removed SW1: MX_SW, PCM_marbastlib-mx:SW_MX_HS_S_CPG151101S11_1u
- PSW1, PSW2: footprint Connector_PinHeader_1.27mm:PinHeader_1x02_P1.27mm_Vertical -> i8:JUMP_1x2; moved to B.Cu
- R3, R5, R6, R7: moved to B.Cu
- moved R3 32.9 mm to (-6.92, 10.1), turned to 45 degrees
- moved R5 31.4 mm to (-8.41, 11.6), turned to -135 degrees
- moved R6 29.9 mm to (-9.73, 12.9), turned to -135 degrees
- moved R7 28.5 mm to (-11.0, 14.2), turned to 45 degrees
- moved PSW2 9.21 mm to (-15.8, 8.79), turned to 135 degrees
- moved PSW1 8.99 mm to (-12.2, 5.25), turned to 135 degrees
Connections:
- J2 pad 2: +3V3 -> SWC
- J2 pad 3: SWC -> SWD
- J2 pad 4: SWD -> RST
- J2 pad 5: RST -> +3V3
Routing:
- net +3V3: track 57.2 -> 52.5 mm
- net Net-(PSW2-Pad2): track 0.00 -> 2.61 mm
- net RST: track 4.28 -> 6.44 mm
- net Net-(R5-Pad2): track 0.00 -> 0.84 mm
- net Q_SEL: track 1.71 -> 2.55 mm
- net SWC: track 5.08 -> 5.60 mm

Commit message: i8 development
Parts:
- removed C13, C14, C15: 1u, Capacitor_SMD:C_0402_1005Metric
- removed J1: ZX-SH1.0-4PWT, Connector_JST:JST_SH_SM04B-SRSS-TB_1x04-1MP_P1.00mm_Horizontal
- removed PSW1: REST, i8:JUMP_1x2
- removed PSW2: BOOT, i8:JUMP_1x2
- removed R3, R5, R6: 5.1k, Resistor_SMD:R_0402_1005Metric
- removed R7: 1k, Resistor_SMD:R_0402_1005Metric
- removed U1: XC6206P332MR-G, Package_TO_SOT_SMD:SOT-23-3
- C1, C10, C11, C12, C16, C17, C2, C3, C4, C5, C6, C7, C8, C9: footprint Capacitor_SMD:C_0402_1005Metric -> i8:C_0402_1005Metric_mod
- moved C2 11.0 mm to (-3.55, -4.28), turned to 135 degrees
- moved C3 11.0 mm to (2.98, 4.85), turned to -45 degrees
- moved C4 1.10 mm to (-6.54, 1.28)
- moved C16 0.95 mm to (8.13, 2.32)
- moved Y1 0.95 mm to (6.61, 3.85)
- moved C17 0.95 mm to (8.42, 5.66)
- moved R4 0.94 mm to (5.06, 5.37)
- moved J2 0.59 mm to (5.08, 6.79)
- moved C9 0.31 mm to (-3.35, 4.48)
- moved C10 0.31 mm to (-5.89, 1.93)
- moved C7 0.31 mm to (4.48, -3.35)
- moved C6 0.31 mm to (1.93, -5.89)
- moved C8 0.24 mm to (3.63, 4.20)
- moved C1 0.24 mm to (-5.33, -2.50)
- moved U3 0.24 mm to (-3.13, -6.28)
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Routing:
- net +3V3: track 52.5 -> 16.1 mm
- net GND: track 29.1 -> 14.0 mm, vias 20 -> 17
- net D-: track 11.6 -> 0.00 mm
- net D+: track 11.3 -> 0.00 mm
- net GPIO15: track 0.00 -> 9.50 mm
- net GPIO14: track 0.00 -> 8.84 mm
- net GPIO16: track 0.00 -> 8.18 mm
- net GPIO13: track 0.00 -> 8.18 mm
- net GPIO12: track 0.00 -> 7.02 mm
- net GPIO17: track 0.00 -> 7.02 mm
- net GPIO5: track 0.00 -> 6.00 mm
- net GPIO11: track 0.00 -> 6.00 mm
- net GPIO6: track 0.00 -> 6.00 mm
- net GPIO29_ADC3: track 0.00 -> 6.00 mm
- net GPIO24: track 0.00 -> 6.00 mm
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Other:
- outline, holes or cut-outs redrawn
- board text added: "copper .9mm"
- board text added: "via"
- board text added: "zone"

Commit message: i8 development
Parts:
- added C13: 1u, i8:C_0402_1005Metric_mod, B.Cu at (-4.16, -23.4)
- added C14: 1u, i8:C_0402_1005Metric_mod, B.Cu at (-6.43, -23.4)
- added C15: 1u, i8:C_0402_1005Metric_mod, B.Cu at (-2.74, -8.35)
- added J1: ZX-SH1.0-4PWT, Connector_JST:JST_SH_SM04B-SRSS-TB_1x04-1MP_P1.00mm_Horizontal, B.Cu at (0.03, -20.0)
- added PSW1: REST, i8:JUMP_REST_10.16mm, F.Cu at (-18.0, 1.75)
- added PSW2: BOOT, i8:JUMP_BOOT_10.16mm, F.Cu at (-18.0, -1.75)
- added R3: 5.1k, Resistor_SMD:R_0402_1005Metric, B.Cu at (-10.8, 2.79)
- added R5: 5.1k, Resistor_SMD:R_0402_1005Metric, B.Cu at (-10.8, 0.93)
- added R6: 5.1k, Resistor_SMD:R_0402_1005Metric, B.Cu at (-10.8, -0.93)
- added R7: 1k, Resistor_SMD:R_0402_1005Metric, B.Cu at (-10.8, -2.79)
- added U1: XC6206P332MR-G, Package_TO_SOT_SMD:SOT-23-3, B.Cu at (-5.29, -21.3)
Routing:
- net +3V3: track 16.1 -> 44.0 mm
- net GND: track 14.0 -> 34.3 mm, vias 17 -> 19
- net D-: track 0.00 -> 18.7 mm
- net D+: track 0.00 -> 16.8 mm
- net +5V: track 0.00 -> 4.64 mm
- net RST: track 5.19 -> 8.09 mm
- net Net-(PSW2-Pad2): track 0.00 -> 2.86 mm
- net Q_SEL: track 1.94 -> 4.14 mm, vias 0 -> 1
- net Net-(R5-Pad2): track 0.00 -> 0.84 mm
