File: 40/i8/i8.kicad_pcb (KiCad board)
At the start: 2 copper layers, 100 x 100 mm, 31 parts, among them J1 ZX-SH1.0-4PWT, J2 Conn_DEBUG, U1 XC6206P332MR-G, U2 RP2040, U3 W25Q16JVUXIQ, Y1 Crystal_GND24

Commit message: tako40_i8 drafted
Parts:
- removed PSW1: REST, Connector_PinHeader_1.27mm:PinHeader_1x02_P1.27mm_Vertical
- removed PSW2: BOOT, Connector_PinHeader_1.27mm:PinHeader_1x02_P1.27mm_Vertical
- removed R3, R5, R6: 5.1k, Resistor_SMD:R_0402_1005Metric
- removed R7: 1k, Resistor_SMD:R_0402_1005Metric
- added C15: 1u, Capacitor_SMD:C_0402_1005Metric, B.Cu at (61.0, 63.9)
- added D1: 1N4148W, Diode_SMD:D_SOD-123, B.Cu at (63.6, 39.0)
- added D10: 1N4148W, Diode_SMD:D_SOD-123, B.Cu at (235.0, 39.0)
- added D11: 1N4148W, Diode_SMD:D_SOD-123, B.Cu at (254.1, 39.0)
- added D12: 1N4148W, Diode_SMD:D_SOD-123, B.Cu at (273.1, 39.0)
- added D13: 1N4148W, Diode_SMD:D_SOD-123, B.Cu at (65.9, 58.0)
- added D14: 1N4148W, Diode_SMD:D_SOD-123, B.Cu at (87.4, 58.0)
- added D15: 1N4148W, Diode_SMD:D_SOD-123, B.Cu at (106.4, 58.0)
- added D16: 1N4148W, Diode_SMD:D_SOD-123, B.Cu at (125.5, 58.0)
- added D17: 1N4148W, Diode_SMD:D_SOD-123, B.Cu at (144.5, 58.0)
- added D18: 1N4148W, Diode_SMD:D_SOD-123, B.Cu at (163.6, 58.0)
- added D19: 1N4148W, Diode_SMD:D_SOD-123, B.Cu at (182.6, 58.0)
- added D2: 1N4148W, Diode_SMD:D_SOD-123, B.Cu at (82.6, 39.0)
- added D20: 1N4148W, Diode_SMD:D_SOD-123, B.Cu at (201.7, 58.0)
- added D21: 1N4148W, Diode_SMD:D_SOD-123, B.Cu at (220.7, 58.0)
- added D22: 1N4148W, Diode_SMD:D_SOD-123, B.Cu at (239.8, 58.0)
- added D23: 1N4148W, Diode_SMD:D_SOD-123, B.Cu at (266.0, 58.0)
- added D24: 1N4148W, Diode_SMD:D_SOD-123, B.Cu at (70.7, 77.1)
- added D25: 1N4148W, Diode_SMD:D_SOD-123, B.Cu at (96.9, 77.1)
- added D26: 1N4148W, Diode_SMD:D_SOD-123, B.Cu at (115.9, 77.1)
- added D27: 1N4148W, Diode_SMD:D_SOD-123, B.Cu at (135.0, 77.1)
- added D28: 1N4148W, Diode_SMD:D_SOD-123, B.Cu at (154.0, 77.1)
- added D29: 1N4148W, Diode_SMD:D_SOD-123, B.Cu at (173.1, 77.1)
- added D3: 1N4148W, Diode_SMD:D_SOD-123, B.Cu at (101.7, 39.0)
- added D30: 1N4148W, Diode_SMD:D_SOD-123, B.Cu at (192.1, 77.1)
- added D31: 1N4148W, Diode_SMD:D_SOD-123, B.Cu at (211.2, 77.1)
- added D32: 1N4148W, Diode_SMD:D_SOD-123, B.Cu at (230.2, 77.1)
- added D33: 1N4148W, Diode_SMD:D_SOD-123, B.Cu at (249.3, 77.1)
- added D34: 1N4148W, Diode_SMD:D_SOD-123, B.Cu at (270.7, 77.1)
- added D35: 1N4148W, Diode_SMD:D_SOD-123, B.Cu at (65.9, 96.1)
- added D36: 1N4148W, Diode_SMD:D_SOD-123, B.Cu at (87.4, 96.1)
- added D37: 1N4148W, Diode_SMD:D_SOD-123, B.Cu at (106.4, 96.1)
- added D38: 1N4148W, Diode_SMD:D_SOD-123, B.Cu at (142.1, 96.1)
- added D4: 1N4148W, Diode_SMD:D_SOD-123, B.Cu at (120.7, 39.0)
- added D41: 1N4148W, Diode_SMD:D_SOD-123, B.Cu at (244.5, 96.1)
- added D42: 1N4148W, Diode_SMD:D_SOD-123, B.Cu at (268.3, 96.1)
- added D44: 1N4148W, Diode_SMD:D_SOD-123, B.Cu at (213.6, 96.1)
- added D47: 1N4148W, Diode_SMD:D_SOD-123, B.Cu at (175.5, 96.1)
- added D5: 1N4148W, Diode_SMD:D_SOD-123, B.Cu at (139.8, 39.0)
- added D6: 1N4148W, Diode_SMD:D_SOD-123, B.Cu at (158.8, 39.0)
- added D7: 1N4148W, Diode_SMD:D_SOD-123, B.Cu at (177.9, 39.0)
- added D8: 1N4148W, Diode_SMD:D_SOD-123, B.Cu at (196.9, 39.0)
- added D9: 1N4148W, Diode_SMD:D_SOD-123, B.Cu at (216.0, 39.0)
- added RV1: RS6011YA600M, shoonies_parts:RS6011YA600M, F.Cu at (43.3, 66.3)
- added S38: MX_S, PCM_marbastlib-mx:STAB_MX_P_2u, B.Cu at (150.5, 94.9)
- added S44: MX_S, PCM_marbastlib-mx:STAB_MX_P_2u, B.Cu at (221.9, 94.9)
- added S47: MX_S, PCM_marbastlib-mx:STAB_MX_P_6.25u, B.Cu at (183.8, 94.9)
- added SW1: MX_SW, PCM_marbastlib-mx:SW_MX_HS_S_CPG151101S11_1u, B.Cu at (71.9, 37.8)
- added SW10: MX_SW, PCM_marbastlib-mx:SW_MX_HS_S_CPG151101S11_1u, B.Cu at (243.3, 37.8)
- added SW11: MX_SW, PCM_marbastlib-mx:SW_MX_HS_S_CPG151101S11_1u, B.Cu at (262.4, 37.8)
- added SW12: MX_SW, PCM_marbastlib-mx:SW_MX_HS_S_CPG151101S11_1u, B.Cu at (281.4, 37.8)
- added SW13: MX_SW, PCM_marbastlib-mx:SW_MX_HS_S_CPG151101S11_1u, B.Cu at (74.3, 56.8)
- added SW14: MX_SW, PCM_marbastlib-mx:SW_MX_HS_S_CPG151101S11_1u, B.Cu at (95.7, 56.8)
- added SW15: MX_SW, PCM_marbastlib-mx:SW_MX_HS_S_CPG151101S11_1u, B.Cu at (114.8, 56.8)
- added SW16: MX_SW, PCM_marbastlib-mx:SW_MX_HS_S_CPG151101S11_1u, B.Cu at (133.8, 56.8)
- added SW17: MX_SW, PCM_marbastlib-mx:SW_MX_HS_S_CPG151101S11_1u, B.Cu at (152.9, 56.8)
- added SW18: MX_SW, PCM_marbastlib-mx:SW_MX_HS_S_CPG151101S11_1u, B.Cu at (171.9, 56.8)
- added SW19: MX_SW, PCM_marbastlib-mx:SW_MX_HS_S_CPG151101S11_1u, B.Cu at (191.0, 56.8)
- added SW2: MX_SW, PCM_marbastlib-mx:SW_MX_HS_S_CPG151101S11_1u, B.Cu at (90.9, 37.8)
- added SW20: MX_SW, PCM_marbastlib-mx:SW_MX_HS_S_CPG151101S11_1u, B.Cu at (210.0, 56.8)
- added SW21: MX_SW, PCM_marbastlib-mx:SW_MX_HS_S_CPG151101S11_1u, B.Cu at (229.1, 56.8)
- added SW22: MX_SW, PCM_marbastlib-mx:SW_MX_HS_S_CPG151101S11_1u, B.Cu at (248.1, 56.8)
- added SW23: MX_SW, PCM_marbastlib-mx:SW_MX_HS_S_CPG151101S11_1u, B.Cu at (274.3, 56.8)
- added SW24: MX_SW, PCM_marbastlib-mx:SW_MX_HS_S_CPG151101S11_1u, B.Cu at (79.0, 75.9)
- added SW25: MX_SW, PCM_marbastlib-mx:SW_MX_HS_S_CPG151101S11_1u, B.Cu at (105.2, 75.9)
- added SW26: MX_SW, PCM_marbastlib-mx:SW_MX_HS_S_CPG151101S11_1u, B.Cu at (124.3, 75.9)
- added SW27: MX_SW, PCM_marbastlib-mx:SW_MX_HS_S_CPG151101S11_1u, B.Cu at (143.3, 75.9)
- added SW28: MX_SW, PCM_marbastlib-mx:SW_MX_HS_S_CPG151101S11_1u, B.Cu at (162.4, 75.9)
- added SW29: MX_SW, PCM_marbastlib-mx:SW_MX_HS_S_CPG151101S11_1u, B.Cu at (181.4, 75.9)
- added SW3: MX_SW, PCM_marbastlib-mx:SW_MX_HS_S_CPG151101S11_1u, B.Cu at (110.0, 37.8)
- added SW30: MX_SW, PCM_marbastlib-mx:SW_MX_HS_S_CPG151101S11_1u, B.Cu at (200.5, 75.9)
- added SW31: MX_SW, PCM_marbastlib-mx:SW_MX_HS_S_CPG151101S11_1u, B.Cu at (219.5, 75.9)
- added SW32: MX_SW, PCM_marbastlib-mx:SW_MX_HS_S_CPG151101S11_1u, B.Cu at (238.6, 75.9)
- added SW33: MX_SW, PCM_marbastlib-mx:SW_MX_HS_S_CPG151101S11_1u, B.Cu at (257.6, 75.9)
- added SW34: MX_SW, PCM_marbastlib-mx:SW_MX_HS_S_CPG151101S11_1u, B.Cu at (279.1, 75.9)
- added SW35: MX_SW, PCM_marbastlib-mx:SW_MX_HS_S_CPG151101S11_1u, B.Cu at (74.3, 94.9)
- added SW36: MX_SW, PCM_marbastlib-mx:SW_MX_HS_S_CPG151101S11_1u, B.Cu at (95.7, 94.9)
- added SW37: MX_SW, PCM_marbastlib-mx:SW_MX_HS_S_CPG151101S11_1u, B.Cu at (114.8, 94.9)
- added SW38: MX_SW, PCM_marbastlib-mx:SW_MX_HS_S_CPG151101S11_1u, B.Cu at (150.5, 94.9)
- added SW4: MX_SW, PCM_marbastlib-mx:SW_MX_HS_S_CPG151101S11_1u, B.Cu at (129.0, 37.8)
- added SW41: MX_SW, PCM_marbastlib-mx:SW_MX_HS_S_CPG151101S11_1u, B.Cu at (252.9, 94.9)
- added SW42: MX_SW, PCM_marbastlib-mx:SW_MX_HS_S_CPG151101S11_1u, B.Cu at (276.7, 94.9)
- added SW43: MX_SW, PCM_marbastlib-mx:SW_MX_HS_S_CPG151101S11_1u, B.Cu at (188.6, 94.9)
- added SW44: MX_SW, PCM_marbastlib-mx:SW_MX_HS_S_CPG151101S11_1u, B.Cu at (221.9, 94.9)
- added SW45: MX_SW, PCM_marbastlib-mx:SW_MX_HS_S_CPG151101S11_1u, B.Cu at (255.2, 94.9)
- added SW46: MX_SW, PCM_marbastlib-mx:SW_MX_HS_S_CPG151101S11_1u, B.Cu at (279.1, 94.9)
- added SW47: MX_SW, PCM_marbastlib-mx:SW_MX_HS_S_CPG151101S11_1u, B.Cu at (183.8, 94.9)
- added SW5: MX_SW, PCM_marbastlib-mx:SW_MX_HS_S_CPG151101S11_1u, B.Cu at (148.1, 37.8)
- added SW6: MX_SW, PCM_marbastlib-mx:SW_MX_HS_S_CPG151101S11_1u, B.Cu at (167.1, 37.8)
- added SW7: MX_SW, PCM_marbastlib-mx:SW_MX_HS_S_CPG151101S11_1u, B.Cu at (186.2, 37.8)
- added SW8: MX_SW, PCM_marbastlib-mx:SW_MX_HS_S_CPG151101S11_1u, B.Cu at (205.2, 37.8)
- added SW9: MX_SW, PCM_marbastlib-mx:SW_MX_HS_S_CPG151101S11_1u, B.Cu at (224.3, 37.8)
- moved J1 101.6 mm to (64.9, 47.3), turned to -90 degrees
- moved C13 94.3 mm to (59.9, 56.9), turned to 135 degrees
- moved C8 93.2 mm to (58.7, 67.6), turned to -45 degrees
- moved U3 93.1 mm to (58.9, 63.5), turned to 45 degrees
- moved C14 92.2 mm to (58.3, 55.3), turned to -45 degrees
- moved U1 91.1 mm to (57.6, 57.7), turned to -45 degrees
- moved R1 90.4 mm to (57.2, 61.0), turned to -135 degrees
- moved C2 90.0 mm to (56.8, 63.2), turned to 45 degrees
- moved C9 89.7 mm to (55.9, 71.1), turned to -45 degrees
- moved R2 89.5 mm to (56.5, 60.3), turned to 45 degrees
- moved C7 89.0 mm to (56.1, 62.5), turned to 45 degrees
- moved C4 87.7 mm to (55.3, 58.8), turned to -45 degrees
- moved C1 87.3 mm to (55.0, 61.4), turned to 45 degrees
- moved C6 86.4 mm to (54.3, 60.7), turned to 45 degrees
- moved C5 85.5 mm to (53.7, 60.1), turned to 45 degrees
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Connections:
- U2 pad 11: GPIO8 -> COL6
- U2 pad 12: GPIO9 -> COL5
- U2 pad 13: GPIO10 -> COL4
- U2 pad 14: GPIO11 -> COL3
- U2 pad 15: GPIO12 -> COL2
- U2 pad 16: GPIO13 -> COL1
- U2 pad 17: GPIO14 -> COL0
- U2 pad 5: GPIO3 -> COL11
- U2 pad 6: GPIO4 -> COL10
- U2 pad 7: GPIO5 -> COL9
- U2 pad 8: GPIO6 -> COL8
- U2 pad 9: GPIO7 -> COL7
Routing:
- net COL10: track 0.00 -> 306.7 mm
- net COL9: track 0.00 -> 283.0 mm
- net COL11: track 0.00 -> 282.0 mm
- net COL8: track 0.00 -> 253.5 mm
- net COL6: track 0.00 -> 221.4 mm
- net COL7: track 0.00 -> 220.7 mm, vias 0 -> 1
- net GPIO0: track 31.2 -> 244.0 mm
- net GPIO15: track 27.1 -> 220.2 mm
- net GPIO2: track 30.5 -> 219.0 mm
- net COL5: track 0.00 -> 187.5 mm, vias 0 -> 1
- net GPIO1: track 30.8 -> 216.9 mm
- net COL3: track 0.00 -> 173.9 mm
- net COL4: track 0.00 -> 172.5 mm, vias 0 -> 1
- net COL2: track 0.00 -> 140.0 mm
- net COL1: track 0.00 -> 122.3 mm
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- added copper zone on B.Cu, net COL11
Other:
- board size 100 x 100 mm -> 252.4 x 76.2 mm
