File: 65/TAKO_i5v6+/TAKO_i5v6+.kicad_pcb (KiCad board)
At the start: 2 copper layers, 323.8 x 95.2 mm, 187 parts, among them J1 ZX-SH1.0-4PWT, J3 Conn_01x05, SW1 MX_SW_solder, SW10 MX_SW_solder, SW11 MX_SW_solder, SW12 MX_SW_solder, SW13 MX_SW_solder, SW15 MX_SW_solder, SW17 MX_SW_solder, SW18 MX_SW_solder, SW19 MX_SW_solder, SW2 MX_SW_solder, SW20 MX_SW_solder, SW21 MX_SW_solder, SW22 MX_SW_solder, SW23 MX_SW_solder, SW24 MX_SW_solder, SW25 MX_SW_solder, SW26 MX_SW_solder, SW27 MX_SW_solder, SW28 MX_SW_solder, SW29 MX_SW_solder, SW3 MX_SW_solder, SW30 MX_SW_solder, SW32 RotaryEncoder_Switch, SW34 MX_SW_solder, SW35 MX_SW_solder, SW36 MX_SW_solder, SW37 MX_SW_solder, SW38 MX_SW_solder, SW39 MX_SW_solder, SW4 MX_SW_solder, SW40 MX_SW_solder, SW41 MX_SW_solder, SW42 MX_SW_solder, SW43 MX_SW_solder, SW44 MX_SW_solder, SW45 MX_SW_solder, SW47 MX_SW_solder, SW48 RotaryEncoder_Switch, SW5 MX_SW_solder, SW50 MX_SW_solder, SW52 MX_SW_solder, SW53 MX_SW_solder, SW54 MX_SW_solder, SW55 MX_SW_solder, SW56 MX_SW_solder, SW57 MX_SW_solder, SW58 MX_SW_solder, SW59 MX_SW_solder, SW6 MX_SW_solder, SW60 MX_SW_solder, SW61 MX_SW_solder, SW62 MX_SW_solder, SW63 MX_SW_solder, SW64 MX_SW_solder, SW65 MX_SW_solder, SW66 MX_SW_solder, SW67 MX_SW_solder, SW68 MX_SW_solder, SW69 MX_SW_solder, SW7 MX_SW_solder, SW70 MX_SW_solder, SW71 MX_SW_solder, SW72 MX_SW_solder, SW73 MX_SW_solder, SW74 MX_SW_solder, SW75 MX_SW_solder, SW76 MX_SW_solder, SW77 MX_SW_solder, SW78 SW_RESET, SW79 SW_BOOTSEL, SW8 MX_SW_solder, SW9 MX_SW_solder, U1 RP2040, U2 XC6206PxxxMR, U4 W25Q128JVS, Y1 Crystal_GND24

Commit message: version label
Parts:
- removed D31, D46: D_Small, shoonies_parts:D_SOD-123_CLEAN
- removed the REF** at (314.3, 95.2)
- removed the REF** at (9.53, 0.00)
- removed the REF** at (161.9, 95.2)
- removed the REF** at (66.7, 95.2)
- removed the REF** at (314.3, 0.00)
- removed the REF** at (238.1, 95.2)
- removed the REF** at (9.53, 95.2)
- removed the REF** at (85.7, 0.00)
- removed the REF** at (161.9, 0.00)
- removed the REF** at (238.1, 0.00)
- added D30: D_Small, shoonies_parts:D_SOD-123_CLEAN, B.Cu at (269.1, 31.0)
- added D47: D_Small, shoonies_parts:D_SOD-123_CLEAN, B.Cu at (261.9, 50.0)
- added REF**: Tab, PCM_kikit:Tab, F.Cu at (323.9, 85.7)
- added REF**: Tab, PCM_kikit:Tab, F.Cu at (0.00, 85.7)
- added REF**: Tab, PCM_kikit:Tab, F.Cu at (323.9, 9.53)
- added REF**: Tab, PCM_kikit:Tab, F.Cu at (0.00, 9.53)
- SW1, SW10, SW11, SW12, SW13, SW15, SW17, SW18, SW19, SW2, SW20, SW21, SW22, SW23, SW24, SW25, SW26, SW27, SW28, SW29, SW3, SW30, SW34, SW35, SW36, SW37, SW38, SW39, SW4, SW40, SW41, SW42, SW43, SW44, SW45, SW47, SW5, SW50, SW52, SW53, SW54, SW55, SW56, SW57, SW58, SW59, SW6, SW60, SW61, SW62, SW63, SW64, SW65, SW66, SW67, SW68, SW69, SW7, SW70, SW71, SW72, SW73, SW74, SW75, SW76, SW77, SW8, SW9: value MX_SW_solder -> SW_MX_HS_S
Routing:
- net ROW0: track 340.2 -> 342.5 mm
