File: chiffre/i8/i8.kicad_pcb (KiCad board)
At the start: 2 copper layers, 238.4 x 88.8 mm, 106 parts, among them J1 ZX-SH1.0-4PWT, J2 Conn_DEBUG, SW1 CPG151101S11, SW10 CPG151101S11, SW11 CPG151101S11, SW12 CPG151101S11, SW13 CPG151101S11, SW14 CPG151101S11, SW15 CPG151101S11, SW16 CPG151101S11, SW17 CPG151101S11, SW18 CPG151101S11, SW19 CPG151101S11, SW2 CPG151101S11, SW20 CPG151101S11, SW21 CPG151101S11, SW22 CPG151101S11, SW23 CPG151101S11, SW24 CPG151101S11, SW25 CPG151101S11, SW26 CPG151101S11, SW27 CPG151101S11, SW28 CPG151101S11, SW29 CPG151101S11, SW3 CPG151101S11, SW30 CPG151101S11, SW31 CPG151101S11, SW32 CPG151101S11, SW33 CPG151101S11, SW34 CPG151101S11, SW4 CPG151101S11, SW5 CPG151101S11, SW6 CPG151101S11, SW7 CPG151101S11, SW8 CPG151101S11, SW9 CPG151101S11, U1 XC6206P332MR-G, U2 RP2040, U3 W25Q16JVUXIQ, Y1 Crystal_GND24

Commit message: version label
Parts:
- added REF**: ToolingHole_1.152mm, MountingHole:ToolingHole_1.152mm, F.Cu at (-75.0, 80.0)
- added REF**: ToolingHole_1.152mm, MountingHole:ToolingHole_1.152mm, F.Cu at (-75.0, -15.0)
- added REF**: mousebites 2mm, PCM_marbastlib-various:mousebites_2mm, B.Cu at (178.3, -7.07)
- added REF**: mousebites 2mm, PCM_marbastlib-various:mousebites_2mm, B.Cu at (186.2, 57.2)
- added REF**: Fiducial_1mm_Mask2mm, Fiducial:Fiducial_1mm_Mask2mm, F.Cu at (208.7, -12.3)
- added REF**: ToolingHole_1.152mm, MountingHole:ToolingHole_1.152mm, F.Cu at (210.0, -15.0)
- added REF**: ToolingHole_1.152mm, MountingHole:ToolingHole_1.152mm, F.Cu at (210.0, 80.0)
- added REF**: Fiducial_1mm_Mask2mm, Fiducial:Fiducial_1mm_Mask2mm, F.Cu at (208.7, 77.3)
- added REF**: Fiducial_1mm_Mask2mm, Fiducial:Fiducial_1mm_Mask2mm, F.Cu at (-73.6, -12.3)
- added REF**: mousebites 2mm, PCM_marbastlib-various:mousebites_2mm, F.Cu at (-51.2, 57.2)
- added REF**: Fiducial_1mm_Mask2mm, Fiducial:Fiducial_1mm_Mask2mm, F.Cu at (-73.6, 77.3)
- added REF**: mousebites 2mm, PCM_marbastlib-various:mousebites_2mm, F.Cu at (-43.3, -7.07)
- PSW1, PSW2: moved to B.Cu
- S17, S33: footprint PCM_marbastlib-mx:STAB_MX_P_2u -> PCM_marbastlib-mx:STAB_MX_2u
- moved C17 96.5 mm to (47.2, 73.2), turned to 173 degrees
- moved C16 93.3 mm to (49.6, 70.9), turned to 83 degrees
- moved J2 92.3 mm to (44.2, 71.3), turned to -142 degrees
- moved Y1 92.1 mm to (47.5, 70.7), turned to 83 degrees
- moved R4 91.0 mm to (45.3, 70.4), turned to -97 degrees
- moved C8 87.7 mm to (45.4, 68.6), turned to -97 degrees
- moved C3 87.3 mm to (44.5, 68.4), turned to -97 degrees
- moved C7 83.2 mm to (51.8, 64.6), turned to -7 degrees
- moved U2 78.4 mm to (46.5, 63.1), turned to 173 degrees
- moved C9 77.4 mm to (40.9, 63.2), turned to 173 degrees
- moved C6 77.3 mm to (52.3, 61.0), turned to -7 degrees
- moved D18 73.1 mm to (128.3, 1.24), turned to 142 degrees
- moved D23 73.1 mm to (130.7, 20.2), turned to 142 degrees
- moved D30 73.1 mm to (114.7, 46.1), turned to 142 degrees
- moved D25 73.1 mm to (112.3, 27.2), turned to 142 degrees
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Connections:
- D1 pad 1: GPIO15 -> GPIO0
- D10 pad 1: GPIO9 -> GPIO1
- D11 pad 1: GPIO8 -> GPIO4
- D12 pad 1: GPIO8 -> GPIO4
- D13 pad 1: GPIO8 -> GPIO4
- D14 pad 1: GPIO8 -> GPIO4
- D15 pad 1: GPIO8 -> GPIO4
- D16 pad 1: GPIO6 -> GPIO19
- D17 pad 1: GPIO6 -> GPIO19
- D18 pad 1: GPIO15 -> GPIO0
- D19 pad 1: GPIO15 -> GPIO0
- D2 pad 1: GPIO15 -> GPIO0
- D20 pad 1: GPIO15 -> GPIO0
- D21 pad 1: GPIO15 -> GPIO0
- D22 pad 1: GPIO15 -> GPIO0
- D23 pad 1: GPIO9 -> GPIO1
- D24 pad 1: GPIO9 -> GPIO1
- D25 pad 1: GPIO9 -> GPIO1
- D26 pad 1: GPIO9 -> GPIO1
- D27 pad 1: GPIO9 -> GPIO1
- D28 pad 1: GPIO8 -> GPIO4
- D29 pad 1: GPIO8 -> GPIO4
- D3 pad 1: GPIO15 -> GPIO0
- D30 pad 1: GPIO8 -> GPIO4
- D31 pad 1: GPIO8 -> GPIO4
- D32 pad 1: GPIO8 -> GPIO4
- D33 pad 1: GPIO6 -> GPIO19
- D34 pad 1: GPIO6 -> GPIO19
- D35 pad 1: GPIO9 -> GPIO1
- D36 pad 1: GPIO6 -> GPIO19
- D4 pad 1: GPIO15 -> GPIO0
- D5 pad 1: GPIO15 -> GPIO0
- D6 pad 1: GPIO9 -> GPIO1
- D7 pad 1: GPIO9 -> GPIO1
- D8 pad 1: GPIO9 -> GPIO1
- D9 pad 1: GPIO9 -> GPIO1
- U2 pad 11: GPIO8 -> COL5
- U2 pad 12: GPIO9 -> COL7
- U2 pad 13: COL4 -> COL9
- U2 pad 14: COL3 -> COL10
- U2 pad 15: COL2 -> COL8
- U2 pad 16: COL1 -> COL6
- U2 pad 17: COL0 -> EC2_B
- U2 pad 18: GPIO15 -> EC2_A
- U2 pad 3: COL5 -> GPIO1
- U2 pad 31: COL10 -> COL2
- U2 pad 32: COL9 -> COL4
- U2 pad 35: COL8 -> COL0
- U2 pad 36: COL7 -> COL1
- U2 pad 37: COL6 -> COL3
- U2 pad 4: EC1_B -> EC1_A
- U2 pad 5: EC1_A -> EC1_B
- U2 pad 6: EC2_B -> GPIO4
- U2 pad 7: EC2_A -> GPIO5
Routing:
- net GPIO8: track 285.8 -> 0.00 mm, vias 2 -> 0
- net GPIO1: track 0.00 -> 285.2 mm, vias 0 -> 2
- net GPIO4: track 0.00 -> 275.2 mm, vias 0 -> 2
- net GPIO9: track 272.4 -> 0.00 mm, vias 3 -> 0
- net GPIO0: track 0.00 -> 271.7 mm
- net GPIO15: track 242.0 -> 0.00 mm, vias 2 -> 0
- net GPIO6: track 237.9 -> 0.00 mm, vias 3 -> 0
- net GPIO19: track 0.00 -> 186.9 mm, vias 0 -> 1
- net RST: track 108.6 -> 18.7 mm, vias 2 -> 1
- net EC2_A: track 85.8 -> 19.8 mm
- net EC2_B: track 90.0 -> 24.0 mm
- net +3V3: track 112.8 -> 53.3 mm, vias 3 -> 1
- net Q_SEL: track 84.7 -> 42.4 mm
- net GND: track 89.3 -> 62.3 mm, vias 23 -> 53
- net COL7: track 100.9 -> 126.3 mm
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- added copper zone on B.Cu, net Net-(PSW2-Pad1)
- added copper zone on F.Cu, net Net-(PSW2-Pad1)
- added copper zone on B.Cu, net RST
- added copper zone on F.Cu, net RST
Other:
- board size 238.4 x 88.8 mm -> 290 x 100 mm
- board text added: "shoonie-desu/zensai_pcb/tree/master/chiffre/i8v2_tako"
- board text removed: "${VERDISPLAY}"
