File: chiffre/i8/i8.kicad_sch (KiCad schematic)
At the start: 106 parts, among them J1 ZX-SH1.0-4PWT, J2 Conn_DEBUG, SW1 CPG151101S11, SW10 CPG151101S11, SW11 CPG151101S11, SW12 CPG151101S11, SW13 CPG151101S11, SW14 CPG151101S11, SW15 CPG151101S11, SW16 CPG151101S11, SW17 CPG151101S11, SW18 CPG151101S11, SW19 CPG151101S11, SW2 CPG151101S11, SW20 CPG151101S11, SW21 CPG151101S11, SW22 CPG151101S11, SW23 CPG151101S11, SW24 CPG151101S11, SW25 CPG151101S11, SW26 CPG151101S11, SW27 CPG151101S11, SW28 CPG151101S11, SW29 CPG151101S11, SW3 CPG151101S11, SW30 CPG151101S11, SW31 CPG151101S11, SW32 CPG151101S11, SW33 CPG151101S11, SW34 CPG151101S11, SW4 CPG151101S11, SW5 CPG151101S11, SW6 CPG151101S11, SW7 CPG151101S11, SW8 CPG151101S11, SW9 CPG151101S11, U1 XC6206P332MR-G, U2 RP2040, U3 W25Q16JVUXIQ, Y1 Crystal_GND24

Commit message: version label
Parts:
- S17, S33: footprint PCM_marbastlib-mx:STAB_MX_P_2u -> PCM_marbastlib-mx:STAB_MX_2u
Connections:
- net COL0: now also U2.35 (GPIO23); no longer U2.17 (GPIO14)
- net COL1: now also U2.36 (GPIO24); no longer U2.16 (GPIO13)
- net COL10: now also U2.14 (GPIO11); no longer U2.31 (GPIO20)
- net COL2: now also U2.31 (GPIO20); no longer U2.15 (GPIO12)
- net COL3: now also U2.37 (GPIO25); no longer U2.14 (GPIO11)
- net COL4: now also U2.32 (GPIO21); no longer U2.13 (GPIO10)
- net COL5: now also U2.11 (GPIO8); no longer U2.3 (GPIO1)
- net COL6: now also U2.16 (GPIO13); no longer U2.37 (GPIO25)
- net COL7: now also U2.12 (GPIO9); no longer U2.36 (GPIO24)
- net COL8: now also U2.15 (GPIO12); no longer U2.35 (GPIO23)
- net COL9: now also U2.13 (GPIO10); no longer U2.32 (GPIO21)
- net EC1_A: now also U2.4 (GPIO2); no longer U2.5 (GPIO3)
- net EC1_B: now also U2.5 (GPIO3); no longer U2.4 (GPIO2)
- net EC2_A: now also U2.18 (GPIO15); no longer U2.7 (GPIO5)
- net EC2_B: now also U2.17 (GPIO14); no longer U2.6 (GPIO4)
- net GPIO0: now also D1.1 (K), D18.1 (K), D19.1 (K), D2.1 (K), D20.1 (K), D21.1 (K), D22.1 (K), D3.1 (K), D4.1 (K), D5.1 (K)
- net GPIO19: now also D16.1 (K), D17.1 (K), D33.1 (K), D34.1 (K), D36.1 (K)
- net GPIO6: no longer D16.1 (K), D17.1 (K), D33.1 (K), D34.1 (K), D36.1 (K)
- removed net GPIO15: D1.1 (K), D18.1 (K), D19.1 (K), D2.1 (K), D20.1 (K), D21.1 (K), D22.1 (K), D3.1 (K), D4.1 (K), D5.1 (K), U2.18 (GPIO15)
- net GPIO8 renamed GPIO4
- net GPIO4: now also U2.6 (GPIO4); no longer U2.11 (GPIO8)
- net GPIO9 renamed GPIO1
- net GPIO1: now also U2.3 (GPIO1); no longer U2.12 (GPIO9)
- new net GPIO5: U2.7 (GPIO5)
Other:
- moved on the sheet: PSW1, PSW2
