File: chiffre/i8/i8v1_tako.kicad_pcb (KiCad board)
At the start: 2 copper layers, 238.4 x 88.8 mm, 106 parts, among them J1 ZX-SH1.0-4PWT, J2 Conn_DEBUG, SW1 CPG151101S11, SW10 CPG151101S11, SW11 CPG151101S11, SW12 CPG151101S11, SW13 CPG151101S11, SW14 CPG151101S11, SW15 CPG151101S11, SW16 CPG151101S11, SW17 CPG151101S11, SW18 CPG151101S11, SW19 CPG151101S11, SW2 CPG151101S11, SW20 CPG151101S11, SW21 CPG151101S11, SW22 CPG151101S11, SW23 CPG151101S11, SW24 CPG151101S11, SW25 CPG151101S11, SW26 CPG151101S11, SW27 CPG151101S11, SW28 CPG151101S11, SW29 CPG151101S11, SW3 CPG151101S11, SW30 CPG151101S11, SW31 CPG151101S11, SW32 CPG151101S11, SW33 CPG151101S11, SW34 CPG151101S11, SW4 CPG151101S11, SW5 CPG151101S11, SW6 CPG151101S11, SW7 CPG151101S11, SW8 CPG151101S11, SW9 CPG151101S11, U1 XC6206P332MR-G, U2 RP2040, U3 W25Q16JVUXIQ, Y1 Crystal_GND24

Commit message: version label
Parts:
- added REF**: Tab, PCM_kikit:Tab, F.Cu at (115.7, 28.0)
- added REF**: Tab, PCM_kikit:Tab, F.Cu at (-115.7, 28.0)
- moved C14 11.6 mm to (16.7, 22.1)
- moved J1 11.6 mm to (14.1, 28.9)
- moved U1 11.6 mm to (14.7, 23.5)
- moved C13 11.6 mm to (17.0, 24.3)
Routing:
- net GND: track 89.3 -> 66.3 mm, vias 23 -> 29
- net D+: track 36.0 -> 24.4 mm
- net D-: track 36.6 -> 24.9 mm
