File: template/i9/i9.kicad_sch (KiCad schematic)
At the start: 1 part, among them U1 RP2350B-QFN80

Commit message: i9 init
Parts:
- removed U1: RP2350B-QFN80, Package_DFN_QFN:QFN-80-1EP_10x10mm_P0.4mm_EP3.4x3.4mm, symbol rp2350b-qfn80:RP2350B-QFN80
- added C1, C11, C17, C18, C19, C20, C21, C22, C23, C24, C8: 100n, Capacitor_SMD:C_0402_1005Metric, symbol Device:C_Small
- added C10, C12, C9: 1u, Capacitor_SMD:C_0402_1005Metric, symbol Device:C_Small
- added C13, C14, C3, C5, C6, C7: 4u7, Capacitor_SMD:C_0402_1005Metric, symbol Device:C_Small
- added C15, C16: 12p, Capacitor_SMD:C_0402_1005Metric, symbol Device:C_Small
- added C2, C4: 10u, symbol Device:C_Polarized_Small
- added D1: BSD3C051V, Diode_SMD:D_SOD-323, symbol Device:D_TVS
- added D2: Schottky, symbol Device:D_Schottky
- added F1: 750 mA, Fuse:Fuse_0603_1608Metric, symbol Device:Fuse_Small
- added J1: UDB, symbol Connector_Generic_MountingPin:Conn_01x04_MountingPin
- added J10, J8, J9: TC2030_SWD, PCM_marbastlib-various:CON_TC2030_outlined, symbol PCM_marbastlib-various:TC2030_SWD
- added J2: HRO_TYPE-C-31-M-14, Connector_USB:USB_C_Receptacle_HRO_TYPE-C-31-M-12, symbol Connector:USB_C_Receptacle_USB2.0
- added J3, J4, J6: Battery, PCM_marbastlib-various:Molex_Pico-EZmate_78171-0002_1x02-1MP_P1.20mm_Vertical, symbol Connector_Generic_MountingPin:Conn_01x02_MountingPin
- added J5, J7: Thermistor, Connector_JST:JST_PH_S2B-PH-K_1x02_P2.00mm_Horizontal, symbol Connector_Generic_MountingPin:Conn_01x02_MountingPin
- added L1, L2: BLM15PX121SN1D, Inductor_SMD:L_0402_1005Metric, symbol Device:L_Small
- added L3: 10 uH, Inductor_SMD:L_0603_1608Metric, symbol Device:L_Small
- added LED1, LED2: orange, LED_SMD:LED_0402_1005Metric, symbol Device:LED_Small
- added LED3, LED4, LED5, LED6, LED7, LED8, LED9: WS2812_2020, PCM_marbastlib-various:LED_WS2812_2020, symbol PCM_marbastlib-various:WS2812_2020
- added Q1, Q3: AO3401A, Package_TO_SOT_SMD:SOT-23, symbol Transistor_FET:AO3401A
- added Q2, Q4: 2N7002, Package_TO_SOT_SMD:SOT-23, symbol Transistor_FET:2N7002
- added R1, R18, R19, R2: 5k1, Resistor_SMD:R_0402_1005Metric, symbol Device:R_Small
- added R10, R12, R5, R6: 1k5, Resistor_SMD:R_0402_1005Metric, symbol Device:R_Small
- added R11: 47k, Resistor_SMD:R_0402_1005Metric, symbol Device:R_Small
- added R13: 3k9, Resistor_SMD:R_0402_1005Metric, symbol Device:R_Small
- added R14, R16, R8: 5k, Resistor_SMD:R_0402_1005Metric, symbol Device:R_Small
- added R15, R24, R4: 100R, Resistor_SMD:R_0402_1005Metric, symbol Device:R_Small
- added R17: 1k, Resistor_SMD:R_0402_1005Metric, symbol Device:R_Small
- added R20: 806k, Resistor_SMD:R_0402_1005Metric, symbol Device:R_Small
- added R21: 2M, Resistor_SMD:R_0402_1005Metric, symbol Device:R_Small
- added R22, R23, R25, R7, R9: 10k, Resistor_SMD:R_0402_1005Metric, symbol Device:R_Small
- added R3: 100k, Resistor_SMD:R_0402_1005Metric, symbol Device:R_Small
- added SW1, SW2: PWR, PCM_marbastlib-various:SW_MSK12C02-HB, symbol Switch:SW_Push_SPDT
- added SW3, SW4, SW5: RST, PCM_marbastlib-various:SW_SPST_SKQG_WithStem, symbol Switch:SW_Push_45deg
- added U1: SRV05-4, Package_TO_SOT_SMD:SOT-23-6, symbol Power_Protection:SRV05-4
- added U10: MAX17048, Package_DFN_QFN:DFN-8-1EP_2x2mm_P0.5mm_EP0.7x1.3mm, symbol marbastlib-various:MAX17048
- added U11: TXB0101, Package_TO_SOT_SMD:SOT-363_SC-70-6_Handsoldering, symbol PCM_marbastlib-various:TXB0101
- added U2: TP4056, Package_SO:SOP-8-1EP_4.57x4.57mm_P1.27mm_EP4.57x4.45mm, symbol PCM_marbastlib-various:TP4056
- added U3: BQ24075, Package_DFN_QFN:VQFN-16-1EP_3x3mm_P0.5mm_EP1.6x1.6mm, symbol Battery_Management:BQ24075RGT
- added U4: DW01A, Package_TO_SOT_SMD:SOT-23-6, symbol PCM_marbastlib-various:DW01A
- added U5: FS8205, Package_TO_SOT_SMD:SOT-23-6, symbol PCM_marbastlib-various:FS8205
- added U6: XC6206PxxxMR, Package_TO_SOT_SMD:SOT-23, symbol Regulator_Linear:XC6206PxxxMR
- added U7: nRF52840_holyiot_18010, PCM_marbastlib-various:nRF52840_holyiot_18010, symbol PCM_marbastlib-various:nRF52840_holyiot_18010
- added U8: nRF52840_moko_mk08, PCM_marbastlib-various:nRF52840_moko_mk08, symbol PCM_marbastlib-various:nRF52840_moko_mk08
- added U9: nRF52840_E73-2G4M08S1C, PCM_marbastlib-various:nRF52840_E73-2G4M08S1C, symbol PCM_marbastlib-various:nRF52840_E73-2G4M08S1C
- added Y1: 32.768 KHz, Crystal:Crystal_SMD_2012-2Pin_2.0x1.2mm, symbol Device:Crystal_Small
Connections:
- new net: LED4.1 (DOUT), LED5.3 (DIN)
- new net: LED3.1 (DOUT), LED4.3 (DIN)
- new net: C15.1, U9.11 (P0.00/XL1), Y1.2
- new net: C16.1, U9.13 (P0.01/XL2), Y1.1
- new net: LED7.1 (DOUT), LED8.3 (DIN)
- new net: LED6.1 (DOUT), LED7.3 (DIN)
- new net: Q4.1 (G), R24.2, R25.1
- new net: F1.1, L1.2
- new net: J2.A5 (CC1), R2.2
- new net: J2.B5 (CC2), R1.2
- new net: Q3.1 (G), Q4.3 (D), R23.2
- new net: R9.1, U3.1 (TS)
- new net: R13.1, U3.16 (ISET)
- new net: R10.2, U3.9 (~{CHG})
- new net: J4.1 (Pin_1), SW2.2 (B)
- new net: LED8.1 (DOUT), LED9.3 (DIN)
- new net: LED2.1 (K), R10.1
- new net: Q2.1 (G), R4.2, R7.1
- new net: R3.1, SW1.1 (A)
- new net: LED1.1 (K), R5.1
- new net: LED5.1 (DOUT), LED6.3 (DIN)
- new net: R22.2, U11.5 (OE)
- new net: R8.1, U2.2 (PROG)
- new net: U4.1 (OD), U5.6 (G1)
- new net: R17.2, U4.2 (CSI)
- new net: U4.3 (OC), U5.4 (G2)
- new net: C8.1, R15.2, U4.5 (VDD)
- new net: C8.2, J6.2 (Pin_2), U4.6 (VSS), U5.1 (S1)
- new net: R5.2, U2.7 (CHRG)
- new net +3.3V: C10.1, C11.1, C12.1, J10.1 (VCC), J8.1 (VCC), J9.1 (VCC), L3.2, R18.2, R19.2, R22.1, U11.1 (VCCA), U6.2 (VO), U7.14 (VDD_nRF), U8.9 (VDD), U9.19 (VDD)
- new net +5V: C13.1, C2.1, C3.1, C5.1, D2.2 (A), F1.2, LED1.2 (A), Q1.1 (G), R14.1, R4.1, R6.1, U1.5 (VP), U2.4 (VCC), U2.8 (CE), U3.13 (IN), U7.22 (VBUS), U8.46 (VBUS), U9.27 (VBUS)
- new net +BATT: C17.2, C4.1, C7.1, J3.1 (Pin_1), J6.1 (Pin_1), Q1.3 (D), R15.1, R3.2, SW2.1 (A), U10.2 (CELL), U10.3 (VDD), U2.5 (BAT), U3.2 (BAT), U3.3 (BAT)
- new net +VSW: C14.1, C6.1, C9.1, D2.1 (K), LED2.2 (A), Q1.2 (S), Q3.2 (S), R20.1, R23.1, U11.6 (VCCB), U3.10 (OUT), U3.11 (OUT), U3.6 (EN1), U6.3 (VI), U8.42 (VDDH), U9.23 (VDDH)
- new net ALERT: U10.5 (~{ALRT})
- new net DCCH: L3.1, U9.25 (DCCH)
- new net Earth: C1.1, D1.2 (A2), J2.A1 (GND), J2.A12 (GND), J2.B1 (GND), J2.B12 (GND), J2.S1 (SHIELD), L2.1
- new net GND: C1.2, C10.2, C11.2, C12.2, C13.2, C14.2, C15.2, C16.2, C17.1, C18.1, C19.1, C2.2, C20.1, C21.1, C22.1, C23.1, C24.1, C3.2, C4.2, C5.2, C6.2, C7.2, C9.2, D1.1 (A1), J1.4 (Pin_4), J1.MP (MountPin), J10.5 (GND), J3.2 (Pin_2), J3.MP (MountPin), J4.2 (Pin_2), J4.MP (MountPin), J5.2 (Pin_2), J5.MP (MountPin), J6.MP (MountPin), J7.2 (Pin_2), J7.MP (MountPin), J8.5 (GND), J9.5 (GND), L2.2, LED3.2 (VSS), LED4.2 (VSS), LED5.2 (VSS), LED6.2 (VSS), LED7.2 (VSS), LED8.2 (VSS), LED9.2 (VSS), Q2.2 (S), Q4.2 (S), R11.2, R12.2, R13.2, R16.2, R17.1, R21.2, R25.2, R6.2, R7.2, R8.2, R9.2, SW1.3 (C), SW3.2, SW4.2, SW5.2, U1.2 (VN), U10.1 (CTG), U10.4 (GND), U10.6 (QSTRT), U10.9 (GND), U11.2 (GND), U2.1 (TEMP), U2.3 (GND), U3.17 (VSS), U3.4 (~{CE}), U3.5 (EN2), U3.8 (VSS), U5.3 (S2), U6.1 (GND), U7.1 (GND), U7.25 (GND), U7.37 (GND), U8.10 (GND), U8.39 (GND), U8.43 (GND), U8.57 (GND), U9.21 (GND), U9.24 (GND), U9.5 (GND)
- new net GNDPWR: R1.1, R2.1
- new net ILIM: R12.1, U3.12 (ILIM)
- new net RST: J10.3 (~{RST}), J8.3 (~{RST}), J9.3 (~{RST}), SW3.1, SW4.1, SW5.1, U7.21 (P0.18-RESET), U8.27 (P0.18-RESET), U9.26 (P0.18/~{RESET})
- new net SCL: R19.1, U10.7 (SCL), U7.13 (P0.05-A), U8.8 (P0.05-A), U9.15 (P0.05/AIN3)
- new net SDA: R18.1, U10.8 (SDA), U7.15 (P0.07), U8.7 (P0.07), U9.22 (P0.07)
- new net SWDCLK: J10.4 (SWCLK), J8.4 (SWCLK), J9.4 (SWCLK), U7.31 (SWDCLK), U8.19 (SWDCLK), U9.39 (SWDCLK)
- new net SWDIO: J10.2 (SWDIO), J8.2 (SWDIO), J9.2 (SWDIO), U7.32 (SWDIO), U8.20 (SWDIO), U9.37 (SWDIO)
- new net SYSOFF: Q2.3 (D), SW1.2 (B), U3.15 (SYSOFF)
- new net TEMP1: J5.1 (Pin_1), J7.1 (Pin_1), R14.2, R16.1
- new net TMR: R11.1, U3.14 (TMR)
- new net UG_EN: R24.1, U7.27 (P1.00), U8.49 (P1.00), U9.36 (P1.00)
- new net UG_HV: LED3.3 (DIN), U11.4 (B)
- new net UG_LV: U11.3 (A), U7.26 (P0.22), U8.31 (P0.22), U9.34 (P0.22)
- new net UG_PWR: C18.2, C19.2, C20.2, C21.2, C22.2, C23.2, C24.2, LED3.4 (VDD), LED4.4 (VDD), LED5.4 (VDD), LED6.4 (VDD), LED7.4 (VDD), LED8.4 (VDD), LED9.4 (VDD), Q3.3 (D)
- new net USB-D+: J1.3 (Pin_3), J2.A6 (D+), J2.B6 (D+), U1.6 (IO4), U7.24 (D+), U8.47 (USB-D-), U9.31 (D+)
- new net USB-D-: J1.2 (Pin_2), J2.A7 (D-), J2.B7 (D-), U1.1 (IO1), U7.23 (D-), U8.48 (USB-D+), U9.29 (D-)
- new net VBUS: J1.1 (Pin_1), J2.A4 (VBUS), J2.A9 (VBUS), J2.B4 (VBUS), J2.B9 (VBUS), L1.1
- new net VSENSE: R20.2, R21.1, U7.11 (P0.31-LF-A)
- new net col0: U7.7 (P0.02-LF-A), U8.2 (P0.02-LF-A), U9.7 (P0.02/AIN0)
- new net col1: U7.8 (P0.28-LF-A), U8.3 (P0.28-LF-A), U9.4 (P0.28/AIN4)
- new net row0: U7.9 (P0.29-LF-A), U8.4 (P0.29-LF-A), U9.8 (P0.29/AIN5)
- new net row1: U7.10 (P0.30-LF-A), U8.5 (P0.30-LF-A), U9.10 (P0.30/AIN6)
- no-connect marks 0 -> 13
Other:
- note added: "Battery Management (Additional considerations)"
- note added: "Battery Management (Simple)"
- note added: "Battery management (advanced)"
- note added: "External DCCH inductor for DC-DC HV input mode"
- note added: "External LF crystal for lower idle power"
- note added: "MCU section (ebyte E73-2G4M08S1C)"
- note added: "MCU section (holyiot 18010)"
- note added: "MCU section (moko MK08a)"
- note added: "Overtemperature protection (BQ24075) Use a 10k thermistor"
- note added: "Overtemperature protection (TP4056) For values of R15/R16 as well as the thermistor, refer to the datasheet."
- note added: "PROG: 5 kOhm -> 250 mA charging current TEMP: Pulled to GND -> no OTP"
- note added: "SYSOFF 1 (SW1 pos 1): Batt OFF SYSOFF 0 (SW1 pos 3): Batt ON"
- note added: "Switch matrix"
- note added: "TMR: (10 x 48 s/kOhm) * 47 kOhm = 22560s = 6.27h ILIM: 1550 AOhm / 1500 Ohm = 1.03 A = 1030 mA ISET: 890 AOhm / 3900 Ohm = 0.228 A = 230 mA EN1: 1, EN2: 0 = 475 mA MAX TS: 10 kOhm to GND = no OTP"
- note added: "USB connectors and protections"
- note added: "Underglow LEDs"
- note added: "Underglow enable"
- note added: "Underglow levelshifter"
- note added: "Voltage sensing (advanced)"
- note added: "Voltage sensing (simple) - Holyiot only!"
- note added: "referenced from: https://github.com/ebastler/zmk-designguide"
