File: chiffre/c8/c8.kicad_pcb (KiCad board)
At the start: 2 copper layers, 290 x 100 mm, 118 parts, among them J1 ZX-SH1.0-4PWT, J2 Conn_DEBUG, SW1 CPG151101S11, SW10 CPG151101S11, SW11 CPG151101S11, SW12 CPG151101S11, SW13 CPG151101S11, SW14 CPG151101S11, SW15 CPG151101S11, SW16 CPG151101S11, SW17 CPG151101S11, SW18 CPG151101S11, SW19 CPG151101S11, SW2 CPG151101S11, SW20 CPG151101S11, SW21 CPG151101S11, SW22 CPG151101S11, SW23 CPG151101S11, SW24 CPG151101S11, SW25 CPG151101S11, SW26 CPG151101S11, SW27 CPG151101S11, SW28 CPG151101S11, SW29 CPG151101S11, SW3 CPG151101S11, SW30 CPG151101S11, SW31 CPG151101S11, SW32 CPG151101S11, SW33 CPG151101S11, SW34 CPG151101S11, SW4 CPG151101S11, SW5 CPG151101S11, SW6 CPG151101S11, SW7 CPG151101S11, SW8 CPG151101S11, SW9 CPG151101S11, U1 XC6206P332MR-G, U2 RP2040, U3 W25Q16JVUXIQ, Y1 Crystal_GND24

Commit message: c8v2 stable
Routing:
- net +3V3: track 53.2 -> 51.8 mm
Other:
- board text added: "shoonie-desu/zensai_pcb/tree/master/chiffre/c8v2_tako"
- board text removed: "shoonie-desu/zensai_pcb/tree/master/chiffre/i8v2_tako"
Changed lines of the file:
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@@
 		(layer "Edge.Cuts")
 	)
-	(gr_text "shoonie-desu/zensai_pcb/tree/master/chiffre/i8v2_tako"
+	(gr_text "shoonie-desu/zensai_pcb/tree/master/chiffre/c8v2_tako"
 		(at -54.253972 64.204185 353)
 		(layer "F.Mask")
@@
 		)
 	)
-	(gr_text "shoonie-desu/zensai_pcb/tree/master/chiffre/i8v2_tako"
+	(gr_text "shoonie-desu/zensai_pcb/tree/master/chiffre/c8v2_tako"
 		(at 181.110622 64.204262 7)
 		(layer "B.Mask")
@@
 	)
 	(segment
-		(start 45.813253 61.824182)
-		(end 45.775036 62.135479)
-		(width 0.2)
-		(layer "B.Cu")
-		(net 3)
-	)
-	(segment
 		(start 38.481627 58.1849)
 		(end 41.790241 55.599929)
@@
 	)
 	(arc
-		(start 46.334401 60.903073)
-		(mid 46.24992 61.159268)
-		(end 46.073827 61.363628)
-		(width 0.2)
-		(layer "B.Cu")
-		(net 3)
-	)
-	(arc
 		(start 36.121478 69.754241)
 		(mid 36.452292 69.729656)
@@
 		(width 0.2)
 		(layer "B.Cu")
-		(net 3)
-	)
-	(arc
-		(start 46.073827 61.363628)
-		(mid 45.897736 61.567988)
-		(end 45.813253 61.824182)
-		(width 0.2)
-		(layer "B.Cu")
