File: chiffre/c8/c8.kicad_pcb (KiCad board)
At the start: 2 copper layers, 263.6 x 92.8 mm, 121 parts, among them J1 ZX-SH1.0-4PWT, J2 Conn_DEBUG, SW1 CPG151101S11, SW10 CPG151101S11, SW11 CPG151101S11, SW12 CPG151101S11, SW13 CPG151101S11, SW14 CPG151101S11, SW15 CPG151101S11, SW16 CPG151101S11, SW17 CPG151101S11, SW18 CPG151101S11, SW19 CPG151101S11, SW2 CPG151101S11, SW20 CPG151101S11, SW21 CPG151101S11, SW22 CPG151101S11, SW23 CPG151101S11, SW24 CPG151101S11, SW25 CPG151101S11, SW26 CPG151101S11, SW27 CPG151101S11, SW28 CPG151101S11, SW29 CPG151101S11, SW3 CPG151101S11, SW30 CPG151101S11, SW31 CPG151101S11, SW32 CPG151101S11, SW33 CPG151101S11, SW34 CPG151101S11, SW35 CPG151101S11, SW36 CPG151101S11, SW37 CPG151101S11, SW38 CPG151101S11, SW4 CPG151101S11, SW5 CPG151101S11, SW6 CPG151101S11, SW7 CPG151101S11, SW8 CPG151101S11, SW9 CPG151101S11, U1 XC6206P332MR-G, U2 RP2040, U3 W25Q16JVUXIQ, Y1 Crystal_GND24

Commit message: c8v3 development
Parts:
- removed the REF** at (-55.3, 59.8)
- removed the REF** at (-47.3, -5.49)
- removed the REF** at (182.2, 59.8)
- removed the REF** at (174.2, -5.49)
- added ?: , , F.Cu at (63.4, 65.7)
- added ?: , , F.Cu at (63.4, 32.4)
- added D41: 1N4148W, c8:D_SOD-123_mod, B.Cu at (55.6, 73.2)
- added REF**: mousebites 2mm, c8:mousebites_2mm, F.Cu at (-55.3, 59.8)
- added REF**: mousebites 2mm, c8:mousebites_2mm, F.Cu at (-47.3, -5.49)
- added REF**: mousebites 2mm, c8:mousebites_2mm, B.Cu at (174.1, -5.49)
- added REF**: mousebites 2mm, c8:mousebites_2mm, B.Cu at (182.1, 59.8)
- added RSW1: SW_Rotary_1x8_MP, c8:alpsalpine_SRBV, F.Cu at (63.4, 65.7)
- moved D39 16.3 mm to (60.9, 17.7), turned to -90 degrees
- moved D16 12.8 mm to (-20.9, 58.7)
- moved D40 12.6 mm to (60.4, 55.6), turned to -90 degrees
- moved J1 9.53 mm to (-26.1, 29.0)
- moved C13 9.53 mm to (-29.8, 25.1)
- moved U1 9.53 mm to (-31.2, 27.1)
- moved C14 9.53 mm to (-32.1, 24.8)
- moved D7 5.55 mm to (-30.3, 21.9)
- turned EC2 to 17 degrees
Connections:
- D1 pad 1: GPIO23 -> GPIO27_ADC1
- D10 pad 1: GPIO24 -> GPIO28_ADC2
- D11 pad 1: GPIO21 -> GPIO26_ADC0
- D12 pad 1: GPIO21 -> GPIO26_ADC0
- D13 pad 1: GPIO21 -> GPIO26_ADC0
- D14 pad 1: GPIO21 -> GPIO26_ADC0
- D15 pad 1: GPIO21 -> GPIO26_ADC0
- D16 pad 1: GPIO15 -> GPIO21
- D18 pad 1: GPIO15 -> GPIO21
- D19 pad 1: GPIO15 -> GPIO21
- D2 pad 1: GPIO23 -> GPIO27_ADC1
- D20 pad 1: GPIO23 -> GPIO27_ADC1
- D21 pad 1: GPIO23 -> GPIO27_ADC1
- D22 pad 1: GPIO23 -> GPIO27_ADC1
- D23 pad 1: GPIO23 -> GPIO27_ADC1
- D24 pad 1: GPIO23 -> GPIO27_ADC1
- D25 pad 1: GPIO24 -> GPIO28_ADC2
- D26 pad 1: GPIO24 -> GPIO28_ADC2
- D27 pad 1: GPIO24 -> GPIO28_ADC2
- D28 pad 1: GPIO24 -> GPIO28_ADC2
- D29 pad 1: GPIO24 -> GPIO28_ADC2
- D3 pad 1: GPIO23 -> GPIO27_ADC1
- D30 pad 1: GPIO21 -> GPIO26_ADC0
- D31 pad 1: GPIO21 -> GPIO26_ADC0
- D32 pad 1: GPIO21 -> GPIO26_ADC0
- D33 pad 1: GPIO21 -> GPIO26_ADC0
- D34 pad 1: GPIO21 -> GPIO26_ADC0
- D36 pad 1: GPIO15 -> GPIO21
- D37 pad 1: GPIO15 -> GPIO21
- D38 pad 1: GPIO15 -> GPIO21
- D39 pad 1: GPIO24 -> GPIO27_ADC1
- D4 pad 1: GPIO23 -> GPIO27_ADC1
- D40 pad 1: GPIO15 -> GPIO26_ADC0
- D5 pad 1: GPIO23 -> GPIO27_ADC1
- D6 pad 1: GPIO24 -> GPIO28_ADC2
- D7 pad 1: GPIO24 -> GPIO28_ADC2
- D8 pad 1: GPIO24 -> GPIO28_ADC2
- D9 pad 1: GPIO24 -> GPIO28_ADC2
- U2 pad 13: EC2_B -> GPIO10
- U2 pad 14: EC2_A -> EC2_B
- U2 pad 15: COL4 -> EC2_A
- U2 pad 16: COL3 -> GPIO13
- U2 pad 17: COL2 -> GPIO14
- U2 pad 29: GPIO18 -> COL4
- U2 pad 30: GPIO19 -> COL3
- U2 pad 31: GPIO20 -> COL2
- U2 pad 37: COL0 -> GPIO25
- U2 pad 41: GPIO29_ADC3 -> COL0
Routing:
- net GPIO28_ADC2: track 0.00 -> 292.8 mm, vias 0 -> 3
- net GPIO23: track 267.1 -> 0.00 mm
- net GPIO27_ADC1: track 0.00 -> 266.6 mm
- net GPIO24: track 252.1 -> 0.00 mm
- net GPIO26_ADC0: track 0.00 -> 250.8 mm, vias 0 -> 5
- net GPIO10: track 0.00 -> 118.1 mm
- net GPIO17: track 0.00 -> 115.8 mm
- net GPIO15: track 209.2 -> 97.6 mm
- net GPIO14: track 0.00 -> 96.3 mm
- net GPIO13: track 0.00 -> 95.4 mm
- net EC2_A: track 96.0 -> 120.5 mm, vias 1 -> 0
- net EC2_B: track 96.4 -> 117.6 mm, vias 1 -> 0
- net GPIO21: track 237.1 -> 216.0 mm, vias 4 -> 1
- net COL3: track 110.6 -> 131.1 mm
- net COL2: track 97.7 -> 115.5 mm, vias 1 -> 0
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