File: chiffre/c8/c8.kicad_pcb (KiCad board)
At the start: 2 copper layers, 263.6 x 92.8 mm, 125 parts, among them J1 ZX-SH1.0-4PWT, J2 Conn_DEBUG, SW1 CPG151101S11, SW10 CPG151101S11, SW11 CPG151101S11, SW12 CPG151101S11, SW13 CPG151101S11, SW14 CPG151101S11, SW15 CPG151101S11, SW16 CPG151101S11, SW17 CPG151101S11, SW18 CPG151101S11, SW19 CPG151101S11, SW2 CPG151101S11, SW20 CPG151101S11, SW21 CPG151101S11, SW22 CPG151101S11, SW23 CPG151101S11, SW24 CPG151101S11, SW25 CPG151101S11, SW26 CPG151101S11, SW27 CPG151101S11, SW28 CPG151101S11, SW29 CPG151101S11, SW3 CPG151101S11, SW30 CPG151101S11, SW31 CPG151101S11, SW32 CPG151101S11, SW33 CPG151101S11, SW34 CPG151101S11, SW35 CPG151101S11, SW36 CPG151101S11, SW37 CPG151101S11, SW38 CPG151101S11, SW4 CPG151101S11, SW5 CPG151101S11, SW6 CPG151101S11, SW7 CPG151101S11, SW8 CPG151101S11, SW9 CPG151101S11, U1 XC6206P332MR-G, U2 RP2040, U3 W25Q16JVUXIQ, Y1 Crystal_GND24

Commit message: finalizing c8v3_tako...
Parts:
- removed ? (x2): , 
- removed the REF** at (-55.3, 59.8)
- removed the REF** at (-47.3, -5.49)
- removed the REF** at (174.1, -5.49)
- removed the REF** at (182.1, 59.8)
- added REF**: mousebites 2mm, c8:mousebites_2mm, F.Cu at (-55.3, 59.8)
- added REF**: mousebites 2mm, c8:mousebites_2mm, F.Cu at (-47.3, -5.49)
- added REF**: mousebites 2mm, c8:mousebites_2mm, B.Cu at (182.2, 59.8)
- added REF**: mousebites 2mm, c8:mousebites_2mm, B.Cu at (174.2, -5.49)
- moved D40 20.1 mm to (53.9, 74.6), turned to 90 degrees
- moved D39 16.3 mm to (53.9, 32.4), turned to 90 degrees
- moved D41 14.1 mm to (53.0, 59.3), turned to -90 degrees
- moved D16 1.33 mm to (-21.7, 59.7), turned to 128 degrees
Connections:
- D1 pad 1: GPIO27_ADC1 -> GPIO23
- D10 pad 1: GPIO28_ADC2 -> GPIO24
- D11 pad 1: GPIO26_ADC0 -> GPIO21
- D12 pad 1: GPIO26_ADC0 -> GPIO21
- D13 pad 1: GPIO26_ADC0 -> GPIO21
- D14 pad 1: GPIO26_ADC0 -> GPIO21
- D15 pad 1: GPIO26_ADC0 -> GPIO21
- D16 pad 1: GPIO21 -> GPIO20
- D18 pad 1: GPIO21 -> GPIO20
- D19 pad 1: GPIO21 -> GPIO20
- D2 pad 1: GPIO27_ADC1 -> GPIO23
- D20 pad 1: GPIO27_ADC1 -> GPIO23
- D21 pad 1: GPIO27_ADC1 -> GPIO23
- D22 pad 1: GPIO27_ADC1 -> GPIO23
- D23 pad 1: GPIO27_ADC1 -> GPIO23
- D24 pad 1: GPIO27_ADC1 -> GPIO23
- D25 pad 1: GPIO28_ADC2 -> GPIO24
- D26 pad 1: GPIO28_ADC2 -> GPIO24
- D27 pad 1: GPIO28_ADC2 -> GPIO24
- D28 pad 1: GPIO28_ADC2 -> GPIO24
- D29 pad 1: GPIO28_ADC2 -> GPIO24
- D3 pad 1: GPIO27_ADC1 -> GPIO23
- D30 pad 1: GPIO26_ADC0 -> GPIO21
- D31 pad 1: GPIO26_ADC0 -> GPIO21
- D32 pad 1: GPIO26_ADC0 -> GPIO21
- D33 pad 1: GPIO26_ADC0 -> GPIO21
- D34 pad 1: GPIO26_ADC0 -> GPIO21
- D36 pad 1: GPIO21 -> GPIO20
- D37 pad 1: GPIO21 -> GPIO20
- D38 pad 1: GPIO21 -> GPIO20
- D39 pad 1: GPIO27_ADC1 -> GPIO24
- D4 pad 1: GPIO27_ADC1 -> GPIO23
- D40 pad 1: GPIO26_ADC0 -> GPIO20
- D40 pad 2: EC2_S2 -> EC2_S1
- D41 pad 1: Net-(D41-K) -> GPIO14
- D41 pad 2: COL5 -> Net-(D41-A)
- D5 pad 1: GPIO27_ADC1 -> GPIO23
- D6 pad 1: GPIO28_ADC2 -> GPIO24
- D7 pad 1: GPIO28_ADC2 -> GPIO24
- D8 pad 1: GPIO28_ADC2 -> GPIO24
- D9 pad 1: GPIO28_ADC2 -> GPIO24
- EC2 pad S1: COL5 -> EC2_S1
- EC2 pad S2: EC2_S2 -> COL5
- RSW1 pad 1: GPIO17 -> COL3
- RSW1 pad 2: GPIO15 -> COL4
- RSW1 pad 3: GPIO14 -> COL5
- RSW1 pad 4: GPIO13 -> COL6
- RSW1 pad 5: GPIO10 -> COL7
- RSW1 pad 6: GPIO21 -> COL8
- RSW1 pad 7: GPIO26_ADC0 -> COL9
- RSW1 pad 8: GPIO28_ADC2 -> COL10
- RSW1 pad C: Net-(D41-K) -> Net-(D41-A)
- U2 pad 13: GPIO10 -> EC2_B
- U2 pad 14: EC2_B -> EC2_A
- U2 pad 15: EC2_A -> COL4
- U2 pad 16: GPIO13 -> COL3
- U2 pad 18: GPIO15 -> COL2
- U2 pad 29: COL4 -> GPIO18
- U2 pad 30: COL3 -> GPIO19
- U2 pad 31: COL2 -> GPIO20
- U2 pad 37: GPIO25 -> COL0
- U2 pad 41: COL0 -> GPIO29_ADC3
Routing:
- net GPIO28_ADC2: track 292.8 -> 0.00 mm, vias 3 -> 0
- net GPIO23: track 0.00 -> 268.1 mm
- net GPIO27_ADC1: track 266.6 -> 0.00 mm
- net GPIO24: track 0.00 -> 256.4 mm, vias 0 -> 2
- net GPIO26_ADC0: track 250.8 -> 0.00 mm, vias 5 -> 0
- net GPIO20: track 0.00 -> 215.0 mm
- net GPIO10: track 118.1 -> 0.00 mm
- net GPIO17: track 115.8 -> 0.00 mm
- net GPIO15: track 97.6 -> 0.00 mm
- net GPIO13: track 95.4 -> 0.00 mm
- net COL10: track 254.9 -> 294.9 mm, vias 1 -> 2
- net COL9: track 234.5 -> 270.8 mm, vias 1 -> 2
- net COL8: track 239.9 -> 272.5 mm, vias 1 -> 2
- net COL5: track 138.4 -> 169.7 mm
- net COL6: track 196.6 -> 227.3 mm, vias 1 -> 2
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