File: chiffre/c8/c8.kicad_sch (KiCad schematic)
At the start: 106 parts, among them J1 ZX-SH1.0-4PWT, J2 Conn_DEBUG, SW1 CPG151101S11, SW10 CPG151101S11, SW11 CPG151101S11, SW12 CPG151101S11, SW13 CPG151101S11, SW14 CPG151101S11, SW15 CPG151101S11, SW16 CPG151101S11, SW17 CPG151101S11, SW18 CPG151101S11, SW19 CPG151101S11, SW2 CPG151101S11, SW20 CPG151101S11, SW21 CPG151101S11, SW22 CPG151101S11, SW23 CPG151101S11, SW24 CPG151101S11, SW25 CPG151101S11, SW26 CPG151101S11, SW27 CPG151101S11, SW28 CPG151101S11, SW29 CPG151101S11, SW3 CPG151101S11, SW30 CPG151101S11, SW31 CPG151101S11, SW32 CPG151101S11, SW33 CPG151101S11, SW34 CPG151101S11, SW4 CPG151101S11, SW5 CPG151101S11, SW6 CPG151101S11, SW7 CPG151101S11, SW8 CPG151101S11, SW9 CPG151101S11, U1 XC6206P332MR-G, U2 RP2040, U3 W25Q16JVUXIQ, Y1 Crystal_GND24

Commit message: finalized chiff c8v2
Parts:
- removed D34: 1N4148W, i8:D_SOD-123_mod, symbol Device:D_45deg
- added D18, D37, D38: 1N4148W, c8:D_SOD-123_mod, symbol Device:D_45deg
- added H1: MountingHole_Pad, MountingHole:MountingHole_3.2mm_M3_Pad_TopBottom, symbol Mechanical:MountingHole_Pad
- added SW18, SW19, SW36, SW37: CPG151101S11, c8:SW_MX_HS_S_CPG151101S11_1u_mod, symbol PCM_marbastlib-mx:MX_SW_solder
- C1, C10, C11, C12, C13, C14, C15, C16, C17, C2, C3, C4, C5, C6, C7, C8, C9: footprint i8:C_0402_1005Metric_mod -> c8:C_0402_1005Metric_mod
- D1, D10, D11, D12, D13, D14, D15, D16, D2, D3, D4, D5, D6, D7, D8, D9: footprint i8:D_SOD-123_mod -> c8:D_SOD-123_mod
- D19: renamed from D17; footprint i8:D_SOD-123_mod -> c8:D_SOD-123_mod
- D20: renamed from D19; footprint i8:D_SOD-123_mod -> c8:D_SOD-123_mod
- D21: renamed from D20; footprint i8:D_SOD-123_mod -> c8:D_SOD-123_mod
- D22: renamed from D18; footprint i8:D_SOD-123_mod -> c8:D_SOD-123_mod
- D23: renamed from D21; footprint i8:D_SOD-123_mod -> c8:D_SOD-123_mod
- D24: renamed from D22; footprint i8:D_SOD-123_mod -> c8:D_SOD-123_mod
- D25: renamed from D24; footprint i8:D_SOD-123_mod -> c8:D_SOD-123_mod
- D26: renamed from D25; footprint i8:D_SOD-123_mod -> c8:D_SOD-123_mod
- D27: renamed from D23; footprint i8:D_SOD-123_mod -> c8:D_SOD-123_mod
- D28: renamed from D26; footprint i8:D_SOD-123_mod -> c8:D_SOD-123_mod
- D29: renamed from D27; footprint i8:D_SOD-123_mod -> c8:D_SOD-123_mod
- D30: renamed from D29; footprint i8:D_SOD-123_mod -> c8:D_SOD-123_mod
- D31: renamed from D30; footprint i8:D_SOD-123_mod -> c8:D_SOD-123_mod
- D32: renamed from D28; footprint i8:D_SOD-123_mod -> c8:D_SOD-123_mod
- D33: renamed from D31; footprint i8:D_SOD-123_mod -> c8:D_SOD-123_mod
- D34: renamed from D32; footprint i8:D_SOD-123_mod -> c8:D_SOD-123_mod
- D36: renamed from D33; footprint i8:D_SOD-123_mod -> c8:D_SOD-123_mod
- D39: renamed from D35; footprint i8:D_SOD-123_mod -> c8:D_SOD-123_mod
- D40: renamed from D36; footprint i8:D_SOD-123_mod -> c8:D_SOD-123_mod
- EC1, EC2: footprint i8:ROT_Alps_EC11E-Switch_mod -> c8:ROT_Alps_EC11E-Switch_mod
- PSW1: footprint i8:JUMP_REST_10.16mm -> c8:JUMP_REST_10.16mm
- PSW2: footprint i8:JUMP_BOOT_10.16mm -> c8:JUMP_BOOT_10.16mm
- SW1, SW10, SW11, SW12, SW13, SW14, SW15, SW16, SW17, SW2, SW3, SW4, SW5, SW6, SW7, SW8, SW9: footprint PCM_marbastlib-mx:SW_MX_HS_S_CPG151101S11_1u -> c8:SW_MX_HS_S_CPG151101S11_1u_mod
- SW20: renamed from SW19; footprint PCM_marbastlib-mx:SW_MX_HS_S_CPG151101S11_1u -> c8:SW_MX_HS_S_CPG151101S11_1u_mod
- SW21: renamed from SW20; footprint PCM_marbastlib-mx:SW_MX_HS_S_CPG151101S11_1u -> c8:SW_MX_HS_S_CPG151101S11_1u_mod
- SW22: renamed from SW18; footprint PCM_marbastlib-mx:SW_MX_HS_S_CPG151101S11_1u -> c8:SW_MX_HS_S_CPG151101S11_1u_mod
- SW23: renamed from SW21; footprint PCM_marbastlib-mx:SW_MX_HS_S_CPG151101S11_1u -> c8:SW_MX_HS_S_CPG151101S11_1u_mod
- SW24: renamed from SW22; footprint PCM_marbastlib-mx:SW_MX_HS_S_CPG151101S11_1u -> c8:SW_MX_HS_S_CPG151101S11_1u_mod
- SW25: renamed from SW24; footprint PCM_marbastlib-mx:SW_MX_HS_S_CPG151101S11_1u -> c8:SW_MX_HS_S_CPG151101S11_1u_mod
- SW26: renamed from SW25; footprint PCM_marbastlib-mx:SW_MX_HS_S_CPG151101S11_1u -> c8:SW_MX_HS_S_CPG151101S11_1u_mod
- SW27: renamed from SW23; footprint PCM_marbastlib-mx:SW_MX_HS_S_CPG151101S11_1u -> c8:SW_MX_HS_S_CPG151101S11_1u_mod
- SW28: renamed from SW26; footprint PCM_marbastlib-mx:SW_MX_HS_S_CPG151101S11_1u -> c8:SW_MX_HS_S_CPG151101S11_1u_mod
- SW29: renamed from SW27; footprint PCM_marbastlib-mx:SW_MX_HS_S_CPG151101S11_1u -> c8:SW_MX_HS_S_CPG151101S11_1u_mod
- SW30: renamed from SW29; footprint PCM_marbastlib-mx:SW_MX_HS_S_CPG151101S11_1u -> c8:SW_MX_HS_S_CPG151101S11_1u_mod
- SW31: renamed from SW30; footprint PCM_marbastlib-mx:SW_MX_HS_S_CPG151101S11_1u -> c8:SW_MX_HS_S_CPG151101S11_1u_mod
- SW32: renamed from SW28; footprint PCM_marbastlib-mx:SW_MX_HS_S_CPG151101S11_1u -> c8:SW_MX_HS_S_CPG151101S11_1u_mod
- SW33: renamed from SW31; footprint PCM_marbastlib-mx:SW_MX_HS_S_CPG151101S11_1u -> c8:SW_MX_HS_S_CPG151101S11_1u_mod
- SW34: renamed from SW32; footprint PCM_marbastlib-mx:SW_MX_HS_S_CPG151101S11_1u -> c8:SW_MX_HS_S_CPG151101S11_1u_mod
- SW35: renamed from SW33; footprint PCM_marbastlib-mx:SW_MX_HS_S_CPG151101S11_1u -> c8:SW_MX_HS_S_CPG151101S11_1u_mod
- SW38: renamed from SW34; footprint PCM_marbastlib-mx:SW_MX_HS_S_CPG151101S11_1u -> c8:SW_MX_HS_S_CPG151101S11_1u_mod
- renumbered S33 to S35
Connections:
- net GPIO5 is gone; now on net COL6: U2.7 (GPIO5)
- net GPIO6 is gone; now on net COL5: U2.8 (GPIO6)
- net COL0: now also U2.37 (GPIO25); no longer U2.35 (GPIO23)
- net COL1: now also U2.2 (GPIO0); no longer U2.36 (GPIO24)
- net COL10: now also U2.3 (GPIO1); no longer U2.14 (GPIO11)
- net COL2: now also U2.17 (GPIO14); no longer U2.31 (GPIO20)
- net COL3: now also U2.16 (GPIO13), SW18.2; no longer U2.37 (GPIO25)
- net COL4: now also SW17.1, U2.15 (GPIO12), SW19.1; no longer SW17.2, U2.32 (GPIO21)
- net COL5: no longer U2.11 (GPIO8)
- net COL6: now also SW21.2, SW26.2, SW31.2, SW36.2; no longer SW20.2, SW25.2, SW30.2, SW35.2, U2.16 (GPIO13)
- net COL7: now also SW22.2, SW27.2, SW32.2, SW35.1, U2.6 (GPIO4), SW37.1; no longer SW21.2, SW26.2, SW31.2, U2.12 (GPIO9)
- net COL8: now also SW20.2, SW25.2, SW30.2, U2.5 (GPIO3); no longer SW22.2, SW27.2, SW32.2, U2.15 (GPIO12)
- net COL9: now also U2.4 (GPIO2); no longer U2.13 (GPIO10)
- net EC1_A: now also U2.12 (GPIO9); no longer U2.4 (GPIO2)
- net EC1_B: now also U2.11 (GPIO8); no longer U2.5 (GPIO3)
- net EC2_A: now also U2.14 (GPIO11); no longer U2.18 (GPIO15)
- net EC2_B: now also U2.13 (GPIO10); no longer U2.17 (GPIO14)
- net GND: now also PSW1.1, PSW2.1, H1.1; no longer PSW1.2, PSW2.2
- net GPIO19: no longer D16.1 (K), D19.1 (K), D36.1 (K), D40.1 (K)
- net RST: now also PSW1.2; no longer PSW1.1
- net at R7.1: now also PSW2.2; no longer PSW2.1
- net at D36.2 (A): now also SW36.1; no longer SW35.1
- net at D19.2 (A): now also SW17.2, SW19.2; no longer SW17.1
- net at SW38.1: now also D38.2 (A)
- net GPIO0 renamed GPIO23
- net GPIO23: now also U2.35 (GPIO23); no longer U2.2 (GPIO0)
- net GPIO1 renamed GPIO24
- net GPIO24: now also U2.36 (GPIO24); no longer U2.3 (GPIO1)
- net GPIO4 renamed GPIO21
- net GPIO21: now also U2.32 (GPIO21); no longer U2.6 (GPIO4)
- new net: D18.2 (A), SW18.1
- new net: D37.2 (A), SW35.2, SW37.2
- new net GPIO15: D16.1 (K), D18.1 (K), D19.1 (K), D36.1 (K), D37.1 (K), D38.1 (K), D40.1 (K), U2.18 (GPIO15)
- new net GPIO20: U2.31 (GPIO20)
Other:
- moved on the sheet: D20, D21, D22, D25, D26, D27, D30, D31, D32, PSW1, PSW2, S17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

Commit message: c8v3 development
Parts:
- added D41: 1N4148W, c8:D_SOD-123_mod, symbol Device:D_45deg
- added RSW1: SW_Rotary_1x8_MP, c8:alpsalpine_SRBV, symbol Switch:SW_Rotary_1x8_MP
Connections:
- net GPIO18 is gone; now on net COL4: U2.29 (GPIO18)
- net GPIO19 is gone; now on net COL3: U2.30 (GPIO19)
- net GPIO20 is gone; now on net COL2: U2.31 (GPIO20)
- net GPIO29_ADC3 is gone; now on net COL0: U2.41 (GPIO29_ADC3)
- net COL0: no longer U2.37 (GPIO25)
- net COL2: no longer U2.17 (GPIO14)
- net COL3: no longer U2.16 (GPIO13)
- net COL4: no longer U2.15 (GPIO12)
- net COL5: now also D41.2 (A)
- net EC2_A: now also U2.15 (GPIO12); no longer U2.14 (GPIO11)
- net EC2_B: now also U2.14 (GPIO11); no longer U2.13 (GPIO10)
- net GND: now also RSW1.MP
- net GPIO15: now also RSW1.2; no longer D16.1 (K), D18.1 (K), D19.1 (K), D36.1 (K), D37.1 (K), D38.1 (K), D40.1 (K)
- net GPIO17: now also RSW1.1
- net GPIO21: now also D16.1 (K), D18.1 (K), D19.1 (K), D36.1 (K), D37.1 (K), D38.1 (K), RSW1.6; no longer D11.1 (K), D12.1 (K), D13.1 (K), D14.1 (K), D15.1 (K), D30.1 (K), D31.1 (K), D32.1 (K), D33.1 (K), D34.1 (K)
- net GPIO23: no longer D1.1 (K), D2.1 (K), D20.1 (K), D21.1 (K), D22.1 (K), D23.1 (K), D24.1 (K), D3.1 (K), D4.1 (K), D5.1 (K)
- net GPIO24: no longer D10.1 (K), D25.1 (K), D26.1 (K), D27.1 (K), D28.1 (K), D29.1 (K), D39.1 (K), D6.1 (K), D7.1 (K), D8.1 (K), D9.1 (K)
- net GPIO26_ADC0: now also D11.1 (K), D12.1 (K), D13.1 (K), D14.1 (K), D15.1 (K), D30.1 (K), D31.1 (K), D32.1 (K), D33.1 (K), D34.1 (K), D40.1 (K), RSW1.7
- net GPIO27_ADC1: now also D1.1 (K), D2.1 (K), D20.1 (K), D21.1 (K), D22.1 (K), D23.1 (K), D24.1 (K), D3.1 (K), D39.1 (K), D4.1 (K), D5.1 (K)
- net GPIO28_ADC2: now also D10.1 (K), D25.1 (K), D26.1 (K), D27.1 (K), D28.1 (K), D29.1 (K), D6.1 (K), D7.1 (K), D8.1 (K), D9.1 (K), RSW1.8
- new net: D41.1 (K), RSW1.C
- new net GPIO10: RSW1.5, U2.13 (GPIO10)
- new net GPIO13: RSW1.4, U2.16 (GPIO13)
- new net GPIO14: RSW1.3, U2.17 (GPIO14)
- new net GPIO25: U2.37 (GPIO25)
Other:
- moved on the sheet: D39, D40
