File: template/c9/c9.kicad_sch (KiCad schematic)
At the start: 95 parts, among them J1 UDB, J10 TC2030_SWD, J2 HRO_TYPE-C-31-M-14, J3 Battery, J4 Battery, J5 Thermistor, J6 Battery, J7 Thermistor, J8 TC2030_SWD, J9 TC2030_SWD, Q1 AO3401A, Q2 2N7002, Q3 AO3401A, Q4 2N7002, SW1 PWR, SW2 PWR, SW3 RST, SW4 RST, SW5 RST, U1 SRV05-4, U10 MAX17048, U11 TXB0101, U2 TP4056, U3 BQ24075, U4 DW01A, U5 FS8205, U6 XC6206PxxxMR, U7 nRF52840_holyiot_18010, U8 nRF52840_moko_mk08, U9 nRF52840_E73-2G4M08S1C, Y1 32.768 KHz

Commit message: c8v2 stable
Parts:
- C1, C10, C11, C12, C13, C14, C15, C16, C17, C18, C19, C20, C21, C22, C23, C24, C3, C5, C6, C7, C8, C9: footprint Capacitor_SMD:C_0402_1005Metric -> c9:C_0402_1005Metric_mod
- J1: footprint (none) -> c9:JST_SH_SM04B-SRSS-TB_1x04-1MP_P1.00mm_Horizontal_mod
- J3: footprint PCM_marbastlib-various:Molex_Pico-EZmate_78171-0002_1x02-1MP_P1.20mm_Vertical -> c9:JST_PH_S2B-PH-SM4-TB_1x02-1MP_P2.00mm_Horizontal_mod
- J9: footprint PCM_marbastlib-various:CON_TC2030_outlined -> Connector_PinHeader_1.00mm:PinHeader_1x05_P1.00mm_Vertical
- LED1, LED2: footprint LED_SMD:LED_0402_1005Metric -> c9:LED_0402_1005Metric_mod
- R1, R10, R11, R12, R13, R14, R15, R16, R17, R18, R19, R2, R20, R21, R22, R23, R24, R25, R3, R4, R5, R6, R7, R8, R9: footprint Resistor_SMD:R_0402_1005Metric -> c9:R_0402_1005Metric_mod
- SW4: footprint PCM_marbastlib-various:SW_SPST_SKQG_WithStem -> c9:JUMP_REST_10.16mm
- U10: footprint Package_DFN_QFN:DFN-8-1EP_2x2mm_P0.5mm_EP0.7x1.3mm -> PCM_Package_DFN_QFN_AKL:DFN-8-1EP_2x2mm_P0.5mm_EP0.7x1.3mm
Connections:
- net +5V: now also J1.1 (Pin_1)
- net VBUS: no longer J1.1 (Pin_1)
- net col0: no longer U8.2 (P0.02-LF-A)
- net col1: no longer U8.3 (P0.28-LF-A)
- net row0: no longer U8.4 (P0.29-LF-A)
- net row1: no longer U8.5 (P0.30-LF-A)
Other:
- moved on the sheet: U8
