File: 60/c8v1/c8v1.kicad_pcb (KiCad board)
At the start: 2 copper layers, 463.4 x 175.3 mm, 188 parts, among them J1 ZX-SH1.0-4PWT, J2 Conn_DEBUG, SW1 CPG151101S11, SW10 CPG151101S11, SW11 CPG151101S11, SW12 CPG151101S11, SW13 CPG151101S11, SW14 CPG151101S11, SW15 CPG151101S11, SW16 CPG151101S11, SW17 CPG151101S11, SW18 CPG151101S11, SW19 CPG151101S11, SW2 CPG151101S11, SW20 CPG151101S11, SW21 CPG151101S11, SW22 CPG151101S11, SW23 CPG151101S11, SW24 CPG151101S11, SW25 CPG151101S11, SW26 CPG151101S11, SW27 CPG151101S11, SW28 CPG151101S11, SW29 CPG151101S11, SW3 CPG151101S11, SW30 CPG151101S11, SW31 CPG151101S11, SW32 CPG151101S11, SW33 CPG151101S11, SW34 CPG151101S11, SW35 CPG151101S11, SW36 CPG151101S11, SW37 CPG151101S11, SW38 CPG151101S11, SW39 CPG151101S11, SW4 CPG151101S11, SW40 CPG151101S11, SW41 CPG151101S11, SW42 CPG151101S11, SW43 CPG151101S11, SW44 CPG151101S11, SW45 CPG151101S11, SW46 CPG151101S11, SW47 CPG151101S11, SW48 CPG151101S11, SW49 CPG151101S11, SW5 CPG151101S11, SW50 CPG151101S11, SW51 CPG151101S11, SW52 CPG151101S11, SW53 CPG151101S11, SW54 CPG151101S11, SW55 CPG151101S11, SW56 CPG151101S11, SW57 CPG151101S11, SW58 CPG151101S11, SW59 CPG151101S11, SW6 CPG151101S11, SW60 CPG151101S11, SW61 CPG151101S11, SW62 CPG151101S11, SW63 CPG151101S11, SW64 CPG151101S11, SW65 CPG151101S11, SW66 CPG151101S11, SW67 CPG151101S11, SW68 CPG151101S11, SW69 CPG151101S11, SW7 CPG151101S11, SW70 CPG151101S11, SW71 CPG151101S11, SW72 CPG151101S11, SW73 CPG151101S11, SW74 CPG151101S11, SW75 CPG151101S11, SW76 CPG151101S11, SW77 CPG151101S11, SW78 CPG151101S11, SW79 CPG151101S11, SW8 CPG151101S11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

Commit message: c8v3_tako finalized
Parts:
- moved D42 30.4 mm to (238.9, 38.1)
- moved D56 25.1 mm to (246.0, 57.1)
- moved D15 22.5 mm to (253.2, 4.85), turned to -90 degrees
- moved D44 14.8 mm to (34.0, 57.1)
- moved D16 14.5 mm to (11.0, 19.1)
- moved D17 14.5 mm to (34.8, 19.1)
- moved D18 14.5 mm to (53.8, 19.1)
- moved D19 14.5 mm to (72.9, 19.1)
- moved D20 14.5 mm to (91.9, 19.1)
- moved D21 14.5 mm to (111.0, 19.1)
- moved D22 14.5 mm to (130.0, 19.1)
- moved D23 14.5 mm to (149.1, 19.1)
- moved D24 14.5 mm to (168.1, 19.1)
- moved D25 14.5 mm to (187.2, 19.1)
- moved D26 14.5 mm to (206.2, 19.1)
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Connections:
- SW14 pad 1: COL14 -> Net-(D15-A)
- SW14 pad 2: Net-(D15-A) -> COL14
- SW16 pad 1: COL14 -> Net-(D15-A)
- SW16 pad 2: Net-(D15-A) -> COL14
- SW45 pad 1: COL13 -> Net-(D42-A)
- SW45 pad 2: Net-(D42-A) -> COL13
- SW46 pad 1: COL13 -> Net-(D42-A)
- SW46 pad 2: Net-(D42-A) -> COL13
- SW49 pad 1: COL1 -> Net-(D44-A)
- SW49 pad 2: Net-(D44-A) -> COL1
- SW60 pad 1: COL14 -> Net-(D56-A)
- SW60 pad 2: Net-(D56-A) -> COL14
Routing:
- net COL14: track 102.4 -> 0.00 mm
- net ROW2: track 263.2 -> 235.7 mm
- net ROW0: track 278.3 -> 258.6 mm
- net ROW3: track 258.5 -> 239.9 mm
- net COL0: track 95.4 -> 77.7 mm
- net COL6: track 100.5 -> 84.8 mm
- net COL13: track 104.3 -> 88.7 mm
- net Net-(D42-A): track 18.9 -> 3.72 mm
- net Net-(D61-A): track 17.9 -> 3.57 mm
- net Net-(D43-A): track 13.1 -> 3.57 mm
- net Net-(D56-A): track 13.1 -> 3.61 mm
- net COL2: track 93.8 -> 85.3 mm
- net COL1: track 91.0 -> 83.5 mm
- net Net-(D59-A): track 14.2 -> 7.01 mm
- net Net-(D58-A): track 11.8 -> 7.01 mm
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Other:
- board size 463.4 x 175.3 mm -> 462.7 x 160.9 mm
