File: 60/c8v1/c8v1.kicad_sch (KiCad schematic)
At the start: 188 parts, among them J1 ZX-SH1.0-4PWT, J2 Conn_DEBUG, SW1 CPG151101S11, SW10 CPG151101S11, SW11 CPG151101S11, SW12 CPG151101S11, SW13 CPG151101S11, SW14 CPG151101S11, SW15 CPG151101S11, SW16 CPG151101S11, SW17 CPG151101S11, SW18 CPG151101S11, SW19 CPG151101S11, SW2 CPG151101S11, SW20 CPG151101S11, SW21 CPG151101S11, SW22 CPG151101S11, SW23 CPG151101S11, SW24 CPG151101S11, SW25 CPG151101S11, SW26 CPG151101S11, SW27 CPG151101S11, SW28 CPG151101S11, SW29 CPG151101S11, SW3 CPG151101S11, SW30 CPG151101S11, SW31 CPG151101S11, SW32 CPG151101S11, SW33 CPG151101S11, SW34 CPG151101S11, SW35 CPG151101S11, SW36 CPG151101S11, SW37 CPG151101S11, SW38 CPG151101S11, SW39 CPG151101S11, SW4 CPG151101S11, SW40 CPG151101S11, SW41 CPG151101S11, SW42 CPG151101S11, SW43 CPG151101S11, SW44 CPG151101S11, SW45 CPG151101S11, SW46 CPG151101S11, SW47 CPG151101S11, SW48 CPG151101S11, SW49 CPG151101S11, SW5 CPG151101S11, SW50 CPG151101S11, SW51 CPG151101S11, SW52 CPG151101S11, SW53 CPG151101S11, SW54 CPG151101S11, SW55 CPG151101S11, SW56 CPG151101S11, SW57 CPG151101S11, SW58 CPG151101S11, SW59 CPG151101S11, SW6 CPG151101S11, SW60 CPG151101S11, SW61 CPG151101S11, SW62 CPG151101S11, SW63 CPG151101S11, SW64 CPG151101S11, SW65 CPG151101S11, SW66 CPG151101S11, SW67 CPG151101S11, SW68 CPG151101S11, SW69 CPG151101S11, SW7 CPG151101S11, SW70 CPG151101S11, SW71 CPG151101S11, SW72 CPG151101S11, SW73 CPG151101S11, SW74 CPG151101S11, SW75 CPG151101S11, SW76 CPG151101S11, SW77 CPG151101S11, SW78 CPG151101S11, SW79 CPG151101S11, SW8 CPG151101S11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

Commit message: c8v3_tako finalized
Connections:
- net COL1: now also SW49.2; no longer SW49.1
- net COL13: now also SW45.2, SW46.2; no longer SW45.1, SW46.1
- net COL14: now also SW14.2, SW16.2, SW60.2; no longer SW14.1, SW16.1, SW60.1
- net at D56.2 (A), SW62.2: now also SW60.1; no longer SW60.2
- net at D44.2 (A): now also SW49.1; no longer SW49.2
- new net: D15.2 (A), SW14.1, SW16.1
- new net: D42.2 (A), SW45.1, SW46.1
Other:
- moved on the sheet: SW14, SW16, SW45, SW46, SW49, SW60
Changed lines of the file:
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@@
 	)
 	(junction
-		(at 309.88 86.36)
-		(diameter 0)
-		(color 0 0 0 0)
-	)
-	(junction
 		(at 91.44 71.12)
 		(diameter 0)
@@
 	)
 	(junction
+		(at 330.2 106.68)
+		(diameter 0)
+		(color 0 0 0 0)
+	)
+	(junction
 		(at 40.64 81.28)
 		(diameter 0)
@@
 	)
 	(junction
-		(at 330.2 45.72)
-		(diameter 0)
-		(color 0 0 0 0)
-	)
-	(junction
 		(at 40.64 40.64)
 		(diameter 0)
@@
 	)
 	(junction
+		(at 309.88 86.36)
+		(diameter 0)
+		(color 0 0 0 0)
+	)
+	(junction
 		(at 45.72 106.68)
 		(diameter 0)
@@
 	)
 	(junction
+		(at 330.2 45.72)
+		(diameter 0)
+		(color 0 0 0 0)
+	)
+	(junction
 		(at 121.92 81.28)
 		(diameter 0)
@@
 	)
 	(junction
-		(at 330.2 106.68)
-		(diameter 0)
-		(color 0 0 0 0)
-	)
-	(junction
 		(at 167.64 127)
 		(diameter 0)
@@
 	(wire
 		(pts
+			(xy 304.8 81.28) (xy 304.8 101.6)
+		)
+		(stroke
+			(width 0)
+			(type default)
+		)
+	)
+	(wire
+		(pts
 			(xy 213.36 50.8) (xy 233.68 50.8)
 		)
@@
 	(wire
 		(pts
-			(xy 304.8 81.28) (xy 304.8 101.6)
-		)
-		(stroke
-			(width 0)
-			(type default)
-		)
-	)
-	(wire
-		(pts
 			(xy 254 111.76) (xy 274.32 111.76)
 		)
@@
 	(symbol
 		(lib_id "PCM_marbastlib-mx:MX_SW_solder")
-		(at 327.66 104.14 0)
+		(at 327.66 104.14 180)
 		(unit 1)
 		(exclude_from_sim no)
@@
 		)
 		(property "Value" "CPG151101S11"
-			(at 327.66 108.2732 0)
+			(at 327.66 100.0068 0)
 			(effects
 				(font
@@
 	(symbol
 		(lib_id "PCM_marbastlib-mx:MX_SW_solder")
-		(at 332.74 43.18 0)
+		(at 332.74 43.18 180)
 		(unit 1)
 		(exclude_from_sim no)
@@
 		)
 		(property "Value" "CPG151101S11"
-			(at 332.74 47.3132 0)
+			(at 332.74 39.0468 0)
 			(effects
 				(font
@@
 	(symbol
 		(lib_id "PCM_marbastlib-mx:MX_SW_solder")
-		(at 327.66 43.18 0)
+		(at 327.66 43.18 180)
 		(unit 1)
 		(exclude_from_sim no)
@@
 		)
 		(property "Value" "CPG151101S11"
-			(at 327.66 47.3132 0)
+			(at 327.66 39.0468 0)
 			(effects
 				(font
@@
 	(symbol
 		(lib_id "PCM_marbastlib-mx:MX_SW_solder")
-		(at 68.58 104.14 0)
+		(at 68.58 104.14 180)
 		(unit 1)
 		(exclude_from_sim no)
@@
 		)
 		(property "Value" "CPG151101S11"
-			(at 68.58 108.2732 0)
+			(at 68.58 100.0068 0)
 			(effects
 				(font
@@
 	(symbol
 		(lib_id "PCM_marbastlib-mx:MX_SW_solder")
-		(at 312.42 83.82 0)
+		(at 312.42 83.82 180)
 		(unit 1)
 		(exclude_from_sim no)
@@
 		)
 		(property "Value" "CPG151101S11"
-			(at 312.42 87.9532 0)
+			(at 312.42 79.6868 0)
 			(effects
 				(font
@@
 	(symbol
 		(lib_id "PCM_marbastlib-mx:MX_SW_solder")
-		(at 307.34 83.82 0)
+		(at 307.34 83.82 180)
 		(unit 1)
 		(exclude_from_sim no)
@@
 		)
 		(property "Value" "CPG151101S11"
-			(at 307.34 87.9532 0)
+			(at 307.34 79.6868 0)
 			(effects
 				(font
