File: chiffre/c10/c10.kicad_pcb (KiCad board)
At the start: 2 copper layers, 263.6 x 92.8 mm, 123 parts, among them J1 ZX-SH1.0-4PWT, J2 Conn_DEBUG, SW1 CPG151101S11, SW10 CPG151101S11, SW11 CPG151101S11, SW12 CPG151101S11, SW13 CPG151101S11, SW14 CPG151101S11, SW15 CPG151101S11, SW16 CPG151101S11, SW17 CPG151101S11, SW18 CPG151101S11, SW19 CPG151101S11, SW2 CPG151101S11, SW20 CPG151101S11, SW21 CPG151101S11, SW22 CPG151101S11, SW23 CPG151101S11, SW24 CPG151101S11, SW25 CPG151101S11, SW26 CPG151101S11, SW27 CPG151101S11, SW28 CPG151101S11, SW29 CPG151101S11, SW3 CPG151101S11, SW30 CPG151101S11, SW31 CPG151101S11, SW32 CPG151101S11, SW33 CPG151101S11, SW34 CPG151101S11, SW35 CPG151101S11, SW36 CPG151101S11, SW37 CPG151101S11, SW38 CPG151101S11, SW4 CPG151101S11, SW5 CPG151101S11, SW6 CPG151101S11, SW7 CPG151101S11, SW8 CPG151101S11, SW9 CPG151101S11, U1 XC6206P332MR-G, U2 RP2040, U3 W25Q16JVUXIQ, Y1 Crystal_GND24

Commit message: c10 drafting
Parts:
- removed C1, C13, C14, C15, C5: 1u, c8:C_0402_1005Metric_mod
- removed C10, C11, C12, C2, C3, C6, C7, C8, C9: 100n, c8:C_0402_1005Metric_mod
- removed C16, C17: 22p, c8:C_0402_1005Metric_mod
- removed C4: 10u, c8:C_0402_1005Metric_mod
- removed D19, D36, D37: 1N4148W, c8:D_SOD-123_mod
- removed J1: ZX-SH1.0-4PWT, Connector_JST:JST_SH_SM04B-SRSS-TB_1x04-1MP_P1.00mm_Horizontal
- removed J2: Conn_DEBUG, Connector_PinHeader_1.27mm:PinHeader_1x05_P1.27mm_Vertical
- removed PSW1: REST, c8:JUMP_REST_10.16mm
- removed PSW2: BOOT, c8:JUMP_BOOT_10.16mm
- removed R1, R2: 27, Resistor_SMD:R_0402_1005Metric
- removed R3, R5, R6: 5.1k, Resistor_SMD:R_0402_1005Metric
- removed R4, R7: 1k, Resistor_SMD:R_0402_1005Metric
- removed REF** (x4): mousebites 2mm, c8:mousebites_2mm
- removed SW18, SW19, SW36, SW37: CPG151101S11, c8:SW_MX_HS_S_CPG151101S11_1u_mod
- removed U1: XC6206P332MR-G, Package_TO_SOT_SMD:SOT-23-3
- removed U2: RP2040, Package_DFN_QFN:QFN-56-1EP_7x7mm_P0.4mm_EP3.2x3.2mm
- removed U3: W25Q16JVUXIQ, Package_SON:Winbond_USON-8-1EP_3x2mm_P0.5mm_EP0.2x1.6mm
- removed Y1: Crystal_GND24, Crystal:Crystal_SMD_3225-4Pin_3.2x2.5mm
- added D17: 1N4148W, c8:D_SOD-123_mod, B.Cu at (-18.5, 212.5)
- added LED1: SK6812, c8:LED_SK6812_PLCC4_5.0x5.0mm_P3.2mm edit, B.Cu at (-42.0, 150.8)
- added LED10: SK6812, c8:LED_SK6812_PLCC4_5.0x5.0mm_P3.2mm edit, B.Cu at (-80.1, 179.4)
- added LED11: SK6812, c8:LED_SK6812_PLCC4_5.0x5.0mm_P3.2mm edit, B.Cu at (-42.0, 188.9)
- added LED12: SK6812, c8:LED_SK6812_PLCC4_5.0x5.0mm_P3.2mm edit, B.Cu at (-61.1, 193.7)
- added LED13: SK6812, c8:LED_SK6812_PLCC4_5.0x5.0mm_P3.2mm edit, B.Cu at (-23.0, 193.7)
- added LED14: SK6812, c8:LED_SK6812_PLCC4_5.0x5.0mm_P3.2mm edit, B.Cu at (-3.94, 193.7)
- added LED15: SK6812, c8:LED_SK6812_PLCC4_5.0x5.0mm_P3.2mm edit, B.Cu at (-80.1, 198.4)
- added LED16: SK6812, c8:LED_SK6812_PLCC4_5.0x5.0mm_P3.2mm edit, B.Cu at (-44.4, 212.7)
- added LED17: SK6812, c8:LED_SK6812_PLCC4_5.0x5.0mm_P3.2mm edit, B.Cu at (-13.5, 212.7)
- added LED2: SK6812, c8:LED_SK6812_PLCC4_5.0x5.0mm_P3.2mm edit, B.Cu at (-61.1, 155.6)
- added LED20: SK6812, c8:LED_SK6812_PLCC4_5.0x5.0mm_P3.2mm edit, B.Cu at (85.1, 135.2)
- added LED21: SK6812, c8:LED_SK6812_PLCC4_5.0x5.0mm_P3.2mm edit, B.Cu at (49.3, 149.0)
- added LED22: SK6812, c8:LED_SK6812_PLCC4_5.0x5.0mm_P3.2mm edit, B.Cu at (67.7, 144.4)
- added LED23: SK6812, c8:LED_SK6812_PLCC4_5.0x5.0mm_P3.2mm edit, B.Cu at (104.7, 135.2)
- added LED24: SK6812, c8:LED_SK6812_PLCC4_5.0x5.0mm_P3.2mm edit, B.Cu at (124.3, 135.2)
- added LED25: SK6812, c8:LED_SK6812_PLCC4_5.0x5.0mm_P3.2mm edit, B.Cu at (89.7, 153.7)
- added LED26: SK6812, c8:LED_SK6812_PLCC4_5.0x5.0mm_P3.2mm edit, B.Cu at (53.9, 167.5)
- added LED27: SK6812, c8:LED_SK6812_PLCC4_5.0x5.0mm_P3.2mm edit, B.Cu at (72.4, 162.9)
- added LED28: SK6812, c8:LED_SK6812_PLCC4_5.0x5.0mm_P3.2mm edit, B.Cu at (109.3, 153.7)
- added LED29: SK6812, c8:LED_SK6812_PLCC4_5.0x5.0mm_P3.2mm edit, B.Cu at (129.0, 153.7)
- added LED3: SK6812, c8:LED_SK6812_PLCC4_5.0x5.0mm_P3.2mm edit, B.Cu at (-23.0, 155.6)
- added LED30: SK6812, c8:LED_SK6812_PLCC4_5.0x5.0mm_P3.2mm edit, B.Cu at (94.3, 172.2)
- added LED31: SK6812, c8:LED_SK6812_PLCC4_5.0x5.0mm_P3.2mm edit, B.Cu at (58.5, 186.0)
- added LED32: SK6812, c8:LED_SK6812_PLCC4_5.0x5.0mm_P3.2mm edit, B.Cu at (77.0, 181.4)
- added LED33: SK6812, c8:LED_SK6812_PLCC4_5.0x5.0mm_P3.2mm edit, B.Cu at (113.9, 172.2)
- added LED34: SK6812, c8:LED_SK6812_PLCC4_5.0x5.0mm_P3.2mm edit, B.Cu at (133.6, 172.2)
- added LED35: SK6812, c8:LED_SK6812_PLCC4_5.0x5.0mm_P3.2mm edit, B.Cu at (72.3, 202.2)
- added LED38: SK6812, c8:LED_SK6812_PLCC4_5.0x5.0mm_P3.2mm edit, B.Cu at (102.4, 194.7)
- added LED4: SK6812, c8:LED_SK6812_PLCC4_5.0x5.0mm_P3.2mm edit, B.Cu at (-3.94, 155.6)
- added LED5: SK6812, c8:LED_SK6812_PLCC4_5.0x5.0mm_P3.2mm edit, B.Cu at (-80.1, 160.3)
- added LED6: SK6812, c8:LED_SK6812_PLCC4_5.0x5.0mm_P3.2mm edit, B.Cu at (-42.0, 169.8)
- added LED7: SK6812, c8:LED_SK6812_PLCC4_5.0x5.0mm_P3.2mm edit, B.Cu at (-61.1, 174.6)
- added LED8: SK6812, c8:LED_SK6812_PLCC4_5.0x5.0mm_P3.2mm edit, B.Cu at (-23.0, 174.6)
- added LED9: SK6812, c8:LED_SK6812_PLCC4_5.0x5.0mm_P3.2mm edit, B.Cu at (-3.94, 174.6)
- moved D5 160.9 mm to (-85.2, 162.4), turned to 90 degrees
- moved D10 160.4 mm to (-85.2, 181.5), turned to 90 degrees
- moved H1 160.1 mm to (-111.5, 141.5), turned to 7 degrees
- moved D15 160.0 mm to (-85.2, 200.5), turned to 90 degrees
- moved D7 158.9 mm to (-66.2, 176.7), turned to 90 degrees
- moved D2 158.7 mm to (-66.2, 157.7), turned to 90 degrees
- moved D12 157.8 mm to (-66.2, 195.8), turned to 90 degrees
- moved H1 156.8 mm to (-100.2, 233.8), turned to 7 degrees
- moved D1 156.6 mm to (-47.1, 152.9), turned to 90 degrees
- moved D6 156.1 mm to (-47.1, 172.0), turned to 90 degrees
- moved SW5 156.0 mm to (-80.1, 155.3), turned to 180 degrees
- moved D11 155.6 mm to (-47.1, 191.0), turned to 90 degrees
- moved SW10 155.6 mm to (-80.1, 174.4), turned to 180 degrees
- moved SW15 155.2 mm to (-80.1, 193.4), turned to 180 degrees
- moved D3 154.2 mm to (-28.1, 157.7), turned to 90 degrees
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Connections:
- net GPIO20 renamed ROW3
- net GPIO21 renamed ROW2
- net GPIO23 renamed ROW0
- net GPIO24 renamed ROW1
- D41 pad 1: GPIO14 -> unconnected-(D41-K-Pad1)
- RSW1 pad 1: COL3 -> unconnected-(RSW1-Pad1)
- RSW1 pad 2: COL4 -> unconnected-(RSW1-Pad2)
- RSW1 pad 3: COL5 -> unconnected-(RSW1-Pad3)
- RSW1 pad 4: COL6 -> unconnected-(RSW1-Pad4)
- RSW1 pad 5: COL7 -> unconnected-(RSW1-Pad5)
- RSW1 pad 6: COL8 -> unconnected-(RSW1-Pad6)
- RSW1 pad 7: COL9 -> unconnected-(RSW1-Pad7)
- RSW1 pad 8: COL10 -> unconnected-(RSW1-Pad8)
- SW17 pad 1: COL4 -> Net-(D17-A)
- SW17 pad 2: Net-(D19-A) -> COL4
- SW35 pad 1: COL7 -> Net-(D18-A)
- SW35 pad 2: Net-(D37-A) -> COL7
Routing:
- net +VLED: track 0.00 -> 467.4 mm, vias 0 -> 1
- net COL10: track 294.9 -> 38.1 mm, vias 2 -> 0
- net COL9: track 270.8 -> 38.1 mm, vias 2 -> 0
- net COL8: track 272.5 -> 63.4 mm, vias 2 -> 0
- net COL7: track 255.1 -> 65.7 mm, vias 2 -> 0
- net COL6: track 227.3 -> 38.1 mm, vias 2 -> 0
- net COL5: track 169.7 -> 0.00 mm, vias 1 -> 0
- net ROW3: track 215.0 -> 53.2 mm
- net EC2_A: track 118.7 -> 0.00 mm
- net EC2_B: track 117.4 -> 0.00 mm
- net COL3: track 154.0 -> 38.1 mm, vias 1 -> 0
- net ROW0: track 268.1 -> 166.4 mm
- net COL4: track 164.1 -> 65.7 mm, vias 1 -> 0
- net EC1_B: track 90.2 -> 0.00 mm
- net ROW1: track 256.4 -> 166.4 mm, vias 2 -> 0
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- removed copper zone on B.Cu, net +1V1
- removed copper zone on F.Cu, net +1V1
- removed copper zone on B.Cu, net +3V3
- removed copper zone on B.Cu, net GND
- removed copper zone on B.Cu, net Net-(PSW2-Pad2)
- removed copper zone on F.Cu, net Net-(PSW2-Pad2)
- removed copper zone on B.Cu, net RST
- removed copper zone on F.Cu, net RST
Other:
- board size 263.6 x 92.8 mm -> 272.5 x 123.9 mm
- board text added: "${REFERENCE}"
- board text removed: "copper .9mm"
- board text removed: "via"
- board text removed: "zone"

Commit message: tag connect routed
Parts:
- added C17: 100n, proj:C_0402_1005Metric, B.Cu at (92.6, 184.5)
- added C25: 12p, proj:C_0402_1005Metric, B.Cu at (96.3, 187.8)
- added C26: 12p, proj:C_0402_1005Metric, B.Cu at (93.2, 185.4)
- added J11: TC2030_SWD, PCM_marbastlib-various:CON_TC2030_outlined, B.Cu at (92.1, 190.7)
- added Q3: AO3401A, Package_TO_SOT_SMD:SOT-23, B.Cu at (48.1, 222.8)
- added Q4: 2N7002, Package_TO_SOT_SMD:SOT-23, B.Cu at (48.1, 227.2)
- added R18: 5k1, proj:R_0402_1005Metric, B.Cu at (92.9, 181.1)
- added R19: 5k1, proj:R_0402_1005Metric, B.Cu at (93.6, 181.6)
- added R22: 10k, proj:R_0402_1005Metric, B.Cu at (44.2, 221.6)
- added R23: 10k, proj:R_0402_1005Metric, B.Cu at (44.2, 223.5)
- added R24: 100R, proj:R_0402_1005Metric, B.Cu at (44.2, 225.4)
- added R25: 10k, proj:R_0402_1005Metric, B.Cu at (44.2, 227.4)
- added U10: MAX17048, Package_DFN_QFN:DFN-8-1EP_2x2mm_P0.5mm_EP0.9x1.3mm, B.Cu at (91.4, 182.6)
- added U11: TXB0101, Package_TO_SOT_SMD:SOT-363_SC-70-6_Handsoldering, B.Cu at (39.8, 222.6)
- added U12: BMD-340-A-R, proj:BMD-340-A-R, B.Cu at (107.7, 188.7)
- added Y2: 32.768 KHz, Crystal:Crystal_SMD_2012-2Pin_2.0x1.2mm, B.Cu at (94.8, 186.5)
- moved H1 42.1 mm to (-131.8, 206.0), turned to 0 degrees
- moved D16 40.5 mm to (-79.2, 193.4), turned to 83 degrees
- moved D15 37.8 mm to (-113.0, 174.8), turned to 83 degrees
- moved LED15 37.2 mm to (-107.7, 173.4), turned to -7 degrees
- moved SW15 36.7 mm to (-107.0, 168.4), turned to 173 degrees
- moved LED16 36.1 mm to (-73.9, 191.9), turned to 173 degrees
- moved D10 36.0 mm to (-110.6, 155.9), turned to 83 degrees
- moved D12 35.9 mm to (-93.5, 172.4), turned to 83 degrees
- moved D18 35.7 mm to (38.4, 198.4), turned to 97 degrees
- moved SW16 35.6 mm to (-73.3, 187.0), turned to 173 degrees
- moved LED10 35.4 mm to (-105.3, 154.5), turned to 173 degrees
- moved LED12 35.3 mm to (-88.2, 171.0), turned to -7 degrees
- moved H1 35.0 mm to (-131.8, 113.0), turned to 0 degrees
- moved SW10 35.0 mm to (-104.7, 149.5), turned to 173 degrees
- moved SW12 34.8 mm to (-87.6, 166.0), turned to 173 degrees
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Connections:
- LED10 pad 2: unconnected-(LED10-DOUT-Pad2) -> Net-(LED10-DOUT)
- LED14 pad 2: unconnected-(LED14-DOUT-Pad2) -> Net-(LED14-DOUT)
- LED15 pad 3: unconnected-(LED15-DIN-Pad3) -> Net-(LED15-DIN)
- LED16 pad 2: unconnected-(LED16-DOUT-Pad2) -> Net-(LED15-DIN)
- LED17 pad 3: unconnected-(LED17-DIN-Pad3) -> Net-(LED17-DIN)
- LED21 pad 3: unconnected-(LED21-DIN-Pad3) -> Net-(LED21-DIN)
- LED26 pad 3: unconnected-(LED26-DIN-Pad3) -> Net-(LED26-DIN)
- LED27 pad 2: Net-(LED25-DIN) -> Net-(LED26-DIN)
- LED27 pad 3: Net-(LED26-DOUT) -> Net-(LED25-DOUT)
- LED28 pad 2: Net-(LED28-DOUT) -> Net-(LED25-DIN)
- LED28 pad 3: Net-(LED25-DOUT) -> Net-(LED28-DIN)
- LED29 pad 2: unconnected-(LED29-DOUT-Pad2) -> Net-(LED28-DIN)
- LED29 pad 3: Net-(LED28-DOUT) -> Net-(LED29-DIN)
- LED31 pad 3: unconnected-(LED31-DIN-Pad3) -> Net-(LED14-DOUT)
- LED34 pad 2: unconnected-(LED34-DOUT-Pad2) -> Net-(LED29-DIN)
- LED35 pad 2: unconnected-(LED35-DOUT-Pad2) -> Net-(LED17-DIN)
- LED4 pad 2: unconnected-(LED4-DOUT-Pad2) -> Net-(LED21-DIN)
- LED5 pad 3: unconnected-(LED5-DIN-Pad3) -> Net-(LED10-DOUT)
- LED9 pad 3: unconnected-(LED9-DIN-Pad3) -> Net-(LED26-DOUT)
Routing:
- net +VLED: track 467.4 -> 749.7 mm, vias 1 -> 28
- net GND: track 185.3 -> 0.00 mm, vias 1 -> 14
- net Net-(LED15-DIN): track 0.00 -> 53.9 mm
- net ROW3: track 53.2 -> 100.0 mm
- net Net-(LED17-DIN): track 0.00 -> 33.9 mm
- net unconnected-(LED17-DIN-Pad3): track 28.8 -> 0.00 mm
- net Net-(LED35-DIN): track 0.00 -> 26.8 mm
- net unconnected-(LED38-DIN-Pad3): track 26.8 -> 0.00 mm
- net Net-(LED16-DIN): track 0.00 -> 26.7 mm
- net Net-(LED29-DIN): track 0.00 -> 26.3 mm
- net Net-(LED10-DOUT): track 0.00 -> 24.4 mm, vias 0 -> 2
- net RST: track 0.00 -> 23.4 mm, vias 0 -> 2
- net SWDIO: track 0.00 -> 23.1 mm, vias 0 -> 2
- net SWDCLK: track 0.00 -> 21.3 mm, vias 0 -> 2
- net Net-(LED6-DIN): track 0.00 -> 17.5 mm
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- added copper zone on B.Cu, net GND
Other:
- board size 272.5 x 123.9 mm -> 263.6 x 92.8 mm
- board text added: "D13"

Commit message: begin matrix signaling
Parts:
- added J1: ZX-SH1.0-6PWT, Connector_JST:JST_SH_SM06B-SRSS-TB_1x06-1MP_P1.00mm_Horizontal, B.Cu at (17.5, 163.1)
- S17, S35: moved to F.Cu
- moved U11 66.3 mm to (97.7, 190.4), turned to -128 degrees
- moved R25 63.4 mm to (95.0, 189.4), turned to 52 degrees
- moved R22 62.7 mm to (97.2, 188.1), turned to -128 degrees
- moved R24 62.5 mm to (95.7, 190.0), turned to -128 degrees
- moved R23 60.9 mm to (94.2, 188.8), turned to 52 degrees
- moved Q4 57.6 mm to (92.9, 191.1), turned to 142 degrees
- moved Q3 56.2 mm to (92.0, 187.8), turned to 142 degrees
- moved J11 19.0 mm to (107.3, 179.3), turned to -38 degrees
- moved C26 0.41 mm to (93.4, 185.1), turned to -128 degrees
- moved C25 0.41 mm to (96.5, 187.5), turned to -128 degrees
- moved U10 0.07 mm to (91.4, 182.6)
- moved R19 0.07 mm to (93.7, 181.6)
- moved R18 0.07 mm to (93.0, 181.0)
- turned S17 to 173 degrees
- turned S35 to -173 degrees
Connections:
- LED38 pad 3: unconnected-(LED38-DIN-Pad3) -> UG_HV
Routing:
- net +VLED: track 749.7 -> 881.6 mm
- net +VSW: track 0.00 -> 127.5 mm, vias 0 -> 3
- net +BATT: track 2.42 -> 116.0 mm, vias 0 -> 2
- net GND: track 0.00 -> 112.1 mm, vias 14 -> 20
- net +5V: track 0.00 -> 107.3 mm
- net USB-D-: track 0.00 -> 107.0 mm
- net USB-D+: track 0.00 -> 106.8 mm
- net ROW3: track 100.0 -> 162.1 mm
- net Net-(LED17-DIN): track 33.9 -> 89.4 mm
- net ROW2: track 176.1 -> 223.0 mm
- net Net-(LED14-DOUT): track 14.9 -> 61.7 mm
- net ROW1: track 181.0 -> 221.3 mm
- net Net-(LED26-DOUT): track 14.9 -> 54.9 mm
- net +3.3V: track 3.88 -> 33.4 mm, vias 1 -> 3
- net SWDCLK: track 21.3 -> 2.15 mm, vias 2 -> 0
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