File: chiffre/c10/c10.kicad_sch (KiCad schematic)
At the start: 115 parts, among them J1 ZX-SH1.0-4PWT, J2 Conn_DEBUG, SW1 CPG151101S11, SW10 CPG151101S11, SW11 CPG151101S11, SW12 CPG151101S11, SW13 CPG151101S11, SW14 CPG151101S11, SW15 CPG151101S11, SW16 CPG151101S11, SW17 CPG151101S11, SW18 CPG151101S11, SW19 CPG151101S11, SW2 CPG151101S11, SW20 CPG151101S11, SW21 CPG151101S11, SW22 CPG151101S11, SW23 CPG151101S11, SW24 CPG151101S11, SW25 CPG151101S11, SW26 CPG151101S11, SW27 CPG151101S11, SW28 CPG151101S11, SW29 CPG151101S11, SW3 CPG151101S11, SW30 CPG151101S11, SW31 CPG151101S11, SW32 CPG151101S11, SW33 CPG151101S11, SW34 CPG151101S11, SW35 CPG151101S11, SW36 CPG151101S11, SW37 CPG151101S11, SW38 CPG151101S11, SW4 CPG151101S11, SW5 CPG151101S11, SW6 CPG151101S11, SW7 CPG151101S11, SW8 CPG151101S11, SW9 CPG151101S11, U1 XC6206P332MR-G, U2 RP2040, U3 W25Q16JVUXIQ, Y1 Crystal_GND24

Commit message: c10 drafting
Parts:
- removed C1, C13, C14, C15, C5: 1u, c8:C_0402_1005Metric_mod, symbol Device:C_Small
- removed C10, C11, C12, C2, C3, C6, C7, C8, C9: 100n, c8:C_0402_1005Metric_mod, symbol Device:C_Small
- removed C16: 22p, c8:C_0402_1005Metric_mod, symbol Device:C_Small
- removed C4: 10u, c8:C_0402_1005Metric_mod, symbol Device:C_Small
- removed D19, D36, D37: 1N4148W, c8:D_SOD-123_mod, symbol Device:D_45deg
- removed J1: ZX-SH1.0-4PWT, Connector_JST:JST_SH_SM04B-SRSS-TB_1x04-1MP_P1.00mm_Horizontal, symbol Connector_Generic_MountingPin:Conn_01x04_MountingPin
- removed J2: Conn_DEBUG, Connector_PinHeader_1.27mm:PinHeader_1x05_P1.27mm_Vertical, symbol Connector_Generic:Conn_01x05
- removed PSW1: REST, c8:JUMP_REST_10.16mm, symbol Switch:SW_Push
- removed PSW2: BOOT, c8:JUMP_BOOT_10.16mm, symbol Switch:SW_Push
- removed R1, R2: 27, Resistor_SMD:R_0402_1005Metric, symbol Device:R_Small
- removed R3, R5, R6: 5.1k, Resistor_SMD:R_0402_1005Metric, symbol Device:R_Small
- removed R4, R7: 1k, Resistor_SMD:R_0402_1005Metric, symbol Device:R_Small
- removed SW18, SW19, SW36, SW37: CPG151101S11, c8:SW_MX_HS_S_CPG151101S11_1u_mod, symbol PCM_marbastlib-mx:MX_SW_solder
- removed U1: XC6206P332MR-G, Package_TO_SOT_SMD:SOT-23-3, symbol Regulator_Linear:XC6206PxxxMR
- removed U2: RP2040, Package_DFN_QFN:QFN-56-1EP_7x7mm_P0.4mm_EP3.2x3.2mm, symbol MCU_RaspberryPi:RP2040
- removed U3: W25Q16JVUXIQ, Package_SON:Winbond_USON-8-1EP_3x2mm_P0.5mm_EP0.2x1.6mm, symbol Memory_Flash:W25Q32JVZP
- removed Y1: Crystal_GND24, Crystal:Crystal_SMD_3225-4Pin_3.2x2.5mm, symbol Device:Crystal_GND24
- added C25, C26: 12p, Capacitor_SMD:C_0402_1005Metric, symbol Device:C_Small
- added D17: 1N4148W, c8:D_SOD-123_mod, symbol Device:D_45deg
- added J11: TC2030_SWD, PCM_marbastlib-various:CON_TC2030_outlined, symbol PCM_marbastlib-various:TC2030_SWD
- added LED1, LED10, LED11, LED12, LED13, LED14, LED15, LED16, LED17, LED2, LED20, LED21, LED22, LED23, LED24, LED25, LED26, LED27, LED28, LED29, LED3, LED30, LED31, LED32, LED33, LED34, LED35, LED38, LED4, LED5, LED6, LED7, LED8, LED9: SK6812, c8:LED_SK6812_PLCC4_5.0x5.0mm_P3.2mm edit, symbol LED:SK6812
- added Q3: AO3401A, Package_TO_SOT_SMD:SOT-23, symbol Transistor_FET:AO3401A
- added Q4: 2N7002, Package_TO_SOT_SMD:SOT-23, symbol Transistor_FET:2N7002
- added R18, R19: 5k1, Resistor_SMD:R_0402_1005Metric, symbol Device:R_Small
- added R22, R23, R25: 10k, Resistor_SMD:R_0402_1005Metric, symbol Device:R_Small
- added R24: 100R, Resistor_SMD:R_0402_1005Metric, symbol Device:R_Small
- added SW18: RST, PCM_marbastlib-various:SW_SPST_SKQG_WithStem, symbol Switch:SW_Push_45deg
- added U10: MAX17048, Package_DFN_QFN:DFN-8-1EP_2x2mm_P0.5mm_EP0.9x1.3mm, symbol marbastlib-various:MAX17048
- added U11: TXB0101, Package_TO_SOT_SMD:SOT-363_SC-70-6_Handsoldering, symbol PCM_marbastlib-various:TXB0101
- added U12: BMD-340-A-R, proj:BMD-340-A-R, symbol proj:BMD-340-A-R
- added Y2: 32.768 KHz, Crystal:Crystal_SMD_2012-2Pin_2.0x1.2mm, symbol Device:Crystal_Small
- C17: value 22p -> 100n; footprint c8:C_0402_1005Metric_mod -> Capacitor_SMD:C_0402_1005Metric; Notes (none) -> X7R, 10%
Connections:
- net +5V: now also U12.66 (VBUS)
- net COL10: no longer RSW1.8
- net COL3: no longer RSW1.1
- net COL4: now also SW17.2; no longer RSW1.2, SW17.1
- net COL5: no longer RSW1.3
- net COL6: no longer RSW1.4
- net COL7: now also SW35.2; no longer RSW1.5, SW35.1
- net COL8: no longer RSW1.6
- net COL9: no longer RSW1.7
- net GND: now also C25.2, C26.2, J11.5 (GND), LED1.4 (VSS), LED10.4 (VSS), LED11.4 (VSS), LED12.4 (VSS), LED13.4 (VSS), LED14.4 (VSS), LED15.4 (VSS), LED16.4 (VSS), LED17.4 (VSS), LED2.4 (VSS), LED20.4 (VSS), LED21.4 (VSS), LED22.4 (VSS), LED23.4 (VSS), LED24.4 (VSS), LED25.4 (VSS), LED26.4 (VSS), LED27.4 (VSS), LED28.4 (VSS), LED29.4 (VSS), LED3.4 (VSS), LED30.4 (VSS), LED31.4 (VSS), LED32.4 (VSS), LED33.4 (VSS), LED34.4 (VSS), LED35.4 (VSS), LED38.4 (VSS), LED4.4 (VSS), LED5.4 (VSS), LED6.4 (VSS), LED7.4 (VSS), LED8.4 (VSS), LED9.4 (VSS), Q4.2 (S), R25.2, SW18.2, U10.1 (CTG), U10.4 (GND), U10.6 (QSTRT), U10.9 (GND), U11.2 (GND), U12.1 (GND), U12.16 (GND), U12.18 (GND), U12.2 (GND), U12.29 (GND), U12.3 (GND), U12.30 (GND), U12.4 (GND), U12.45 (GND), U12.46 (GND), U12.47 (GND), U12.5 (GND), U12.55 (GND)
- net RST: now also J11.3 (~{RST}), SW18.1, U12.39 (P0.18/~{RESET})
- net at D18.2 (A): now also SW35.1
- net +BATT: now reaches C17.2
- net +BATT: now also U10.2 (CELL), U10.3 (VDD)
- net GPIO14: no longer names the net of D41.1 (K)
- net GPIO20 renamed ROW3
- net ROW3: now also D17.1 (K)
- net GPIO21 renamed ROW2
- net GPIO23 renamed ROW0
- net GPIO24 renamed ROW1
- new net: LED25.2 (DOUT), LED28.3 (DIN)
- new net: LED25.3 (DIN), LED27.2 (DOUT)
- new net: LED3.2 (DOUT), LED4.3 (DIN)
- new net: LED1.2 (DOUT), LED3.3 (DIN)
- new net: LED35.3 (DIN), LED38.2 (DOUT)
- new net: LED1.3 (DIN), LED2.2 (DOUT)
- new net: LED2.3 (DIN), LED5.2 (DOUT)
- new net: LED28.2 (DOUT), LED29.3 (DIN)
- new net: LED16.3 (DIN), LED17.2 (DOUT)
- new net: LED30.2 (DOUT), LED33.3 (DIN)
- new net: LED30.3 (DIN), LED32.2 (DOUT)
- new net: LED10.3 (DIN), LED7.2 (DOUT)
- new net: LED31.2 (DOUT), LED32.3 (DIN)
- new net: Q4.1 (G), R24.2, R25.1
- new net: LED26.2 (DOUT), LED27.3 (DIN)
- new net: LED6.3 (DIN), LED8.2 (DOUT)
- new net: LED8.3 (DIN), LED9.2 (DOUT)
- new net: Q3.1 (G), Q4.3 (D), R23.2
- new net: LED20.2 (DOUT), LED23.3 (DIN)
- new net: LED20.3 (DIN), LED22.2 (DOUT)
- new net: LED21.2 (DOUT), LED22.3 (DIN)
- new net: C26.1, U12.14 (XL2/P0.01), Y2.1
- new net: C25.1, U12.13 (XL1/P0.00), Y2.2
- new net: LED6.2 (DOUT), LED7.3 (DIN)
- new net: LED33.2 (DOUT), LED34.3 (DIN)
- new net: LED23.2 (DOUT), LED24.3 (DIN)
- new net: LED13.2 (DOUT), LED14.3 (DIN)
- new net: LED11.3 (DIN), LED12.2 (DOUT)
- new net: LED12.3 (DIN), LED15.2 (DOUT)
- new net: D17.2 (A), SW17.1
- new net: R22.2, U11.5 (OE)
- new net: LED11.2 (DOUT), LED13.3 (DIN)
- new net +3.3V: J11.1 (VCC), R18.2, R19.2, R22.1, U11.1 (VCCA), U12.17 (VCC)
- new net +VLED: LED1.1 (VDD), LED10.1 (VDD), LED11.1 (VDD), LED12.1 (VDD), LED13.1 (VDD), LED14.1 (VDD), LED15.1 (VDD), LED16.1 (VDD), LED17.1 (VDD), LED2.1 (VDD), LED20.1 (VDD), LED21.1 (VDD), LED22.1 (VDD), LED23.1 (VDD), LED24.1 (VDD), LED25.1 (VDD), LED26.1 (VDD), LED27.1 (VDD), LED28.1 (VDD), LED29.1 (VDD), LED3.1 (VDD), LED30.1 (VDD), LED31.1 (VDD), LED32.1 (VDD), LED33.1 (VDD), LED34.1 (VDD), LED35.1 (VDD), LED38.1 (VDD), LED4.1 (VDD), LED5.1 (VDD), LED6.1 (VDD), LED7.1 (VDD), LED8.1 (VDD), LED9.1 (VDD), Q3.3 (D)
- new net +VSW: Q3.2 (S), R23.1, U11.6 (VCCB), U12.65 (VCCH)
- new net ALERT: U10.5 (~{ALRT})
- new net SCL: R19.1, U10.7 (SCL), U12.21 (AIN3/P0.05)
- new net SDA: R18.1, U10.8 (SDA), U12.23 (TRACECLK/P0.07)
- new net SWDCLK: J11.4 (SWCLK), U12.43 (SWCLK)
- new net SWDIO: J11.2 (SWDIO), U12.44 (SWDIO)
- new net UG_EN: R24.1, U12.56 (TRACEDATA0/P1.00)
- new net UG_HV: U11.4 (B)
- new net UG_LV: U11.3 (A), U12.40 (P0.22)
- new net USB-D+: U12.68 (D+)
- new net USB-D-: U12.67 (D-)
- no-connect marks 0 -> 1
Other:
- note added: "Underglow enable"
- note added: "Underglow levelshifter"
- note added: "Voltage sensing (advanced)"
- note added: "controller module"
- moved on the sheet: D1, D10, D11, D12, D13, D14, D15, D16, D2, D20, D21, D22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

Commit message: tag connect routed
Parts:
- C17, C25, C26: footprint Capacitor_SMD:C_0402_1005Metric -> proj:C_0402_1005Metric
- H1: footprint MountingHole:MountingHole_3.2mm_M3_Pad_TopBottom -> proj:standoff
- R18, R19, R22, R23, R24, R25: footprint Resistor_SMD:R_0402_1005Metric -> proj:R_0402_1005Metric
Connections:
- net at LED25.2 (DOUT): now also LED27.3 (DIN); no longer LED28.3 (DIN)
- net at LED25.3 (DIN): now also LED28.2 (DOUT); no longer LED27.2 (DOUT)
- net at LED29.2 (DOUT): now also LED28.3 (DIN)
- net at LED29.3 (DIN): now also LED34.2 (DOUT); no longer LED28.2 (DOUT)
- net at LED16.2 (DOUT): now also LED15.3 (DIN)
- net at LED10.2 (DOUT): now also LED5.3 (DIN)
- net at LED31.3 (DIN): now also LED14.2 (DOUT)
- net at LED26.2 (DOUT): now also LED9.3 (DIN); no longer LED27.3 (DIN)
- net at LED4.2 (DOUT): now also LED21.3 (DIN)
- net at LED17.3 (DIN): now also LED35.2 (DOUT)
- net at LED26.3 (DIN): now also LED27.2 (DOUT)
- no-connect marks 1 -> 2
Changed lines of the file:
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@@
 		(at 252.73 87.63)
 	)
+	(no_connect
+		(at 203.2 130.81)
+	)
+	(wire
+		(pts
+			(xy 100.33 176.53) (xy 127 176.53)
+		)
+		(stroke
+			(width 0)
+			(type default)
+		)
+	)
 	(wire
 		(pts
@@
 	(wire
 		(pts
+			(xy 203.2 153.67) (xy 203.2 176.53)
+		)
+		(stroke
+			(width 0)
+			(type default)
+		)
+	)
+	(wire
+		(pts
 			(xy 347.98 130.81) (xy 347.98 139.7)
 		)
@@
 	(wire
 		(pts
+			(xy 100.33 130.81) (xy 127 130.81)
+		)
+		(stroke
+			(width 0)
+			(type default)
+		)
+	)
+	(wire
+		(pts
 			(xy 72.39 83.82) (xy 87.63 83.82)
 		)
@@
 	(wire
 		(pts
+			(xy 24.13 130.81) (xy 24.13 153.67)
+		)
+		(stroke
+			(width 0)
+			(type default)
+		)
+	)
+	(wire
+		(pts
 			(xy 133.35 83.82) (xy 148.59 83.82)
 		)
@@
 	(wire
 		(pts
+			(xy 54.61 199.39) (xy 24.13 199.39)
+		)
+		(stroke
+			(width 0)
+			(type default)
+		)
+	)
+	(wire
+		(pts
+			(xy 100.33 199.39) (xy 127 199.39)
+		)
+		(stroke
+			(width 0)
+			(type default)
+		)
+	)
+	(wire
+		(pts
 			(xy 87.63 83.82) (xy 102.87 83.82)
 		)
@@
 	(wire
 		(pts
+			(xy 24.13 199.39) (xy 24.13 176.53)
+		)
+		(stroke
+			(width 0)
+			(type default)
+		)
+	)
+	(wire
+		(pts
 			(xy 118.11 99.06) (xy 148.59 99.06)
 		)
@@
 	(wire
 		(pts
+			(xy 100.33 153.67) (xy 127 153.67)
+		)
+		(stroke
+			(width 0)
+			(type default)
+		)
+	)
+	(wire
+		(pts
 			(xy 386.08 62.23) (xy 388.62 62.23)
 		)
@@
 		(lib_id "LED:SK6812")
 		(at 165.1 153.67 0)
+		(mirror y)
 		(unit 1)
 		(exclude_from_sim no)
@@
 		(dnp no)
 		(property "Reference" "LED25"
-			(at 162.052 147.32 0)
+			(at 168.148 147.32 0)
 			(effects
 				(font
@@
 		)
 		(property "Value" "SK6812"
-			(at 175.26 149.7898 0)
+			(at 154.94 149.7898 0)
 			(effects
 				(font
@@
 		)
 		(property "Footprint" "c8:LED_SK6812_PLCC4_5.0x5.0mm_P3.2mm edit"
-			(at 166.37 161.29 0)
+			(at 163.83 161.29 0)
 			(effects
 				(font
@@
 		)
 		(property "Datasheet" "https://cdn-shop.adafruit.com/product-files/1138/SK6812+LED+datasheet+.pdf"
-			(at 167.64 163.195 0)
+			(at 162.56 163.195 0)
 			(effects
 				(font
@@
 		(lib_id "LED:SK6812")
 		(at 195.58 153.67 0)
+		(mirror y)
 		(unit 1)
 		(exclude_from_sim no)
@@
 		(dnp no)
 		(property "Reference" "LED29"
-			(at 192.532 147.32 0)
+			(at 198.628 147.32 0)
 			(effects
 				(font
@@
 		)
 		(property "Value" "SK6812"
-			(at 205.74 149.7898 0)
+			(at 185.42 149.7898 0)
 			(effects
 				(font
@@
 		)
 		(property "Footprint" "c8:LED_SK6812_PLCC4_5.0x5.0mm_P3.2mm edit"
-			(at 196.85 161.29 0)
+			(at 194.31 161.29 0)
 			(effects
 				(font
@@
 		)
 		(property "Datasheet" "https://cdn-shop.adafruit.com/product-files/1138/SK6812+LED+datasheet+.pdf"
-			(at 198.12 163.195 0)
+			(at 193.04 163.195 0)
 			(effects
 				(font
@@
 			)
 		)
-		(property "Footprint" "Resistor_SMD:R_0402_1005Metric"
+		(property "Footprint" "proj:R_0402_1005Metric"
 			(at 353.06 105.41 0)
 			(effects
@@
 		(lib_id "LED:SK6812")
 		(at 149.86 153.67 0)
+		(mirror y)
 		(unit 1)
 		(exclude_from_sim no)
@@
 		(dnp no)
 		(property "Reference" "LED27"
-			(at 146.812 147.32 0)
+			(at 152.908 147.32 0)
 			(effects
 				(font
@@
 		)
 		(property "Value" "SK6812"
-			(at 160.02 149.7898 0)
+			(at 139.7 149.7898 0)
 			(effects
 				(font
@@
 		)
 		(property "Footprint" "c8:LED_SK6812_PLCC4_5.0x5.0mm_P3.2mm edit"
-			(at 151.13 161.29 0)
+			(at 148.59 161.29 0)
 			(effects
 				(font
@@
 		)
 		(property "Datasheet" "https://cdn-shop.adafruit.com/product-files/1138/SK6812+LED+datasheet+.pdf"
-			(at 152.4 163.195 0)
+			(at 147.32 163.195 0)
 			(effects
 				(font
@@
 			)
 		)
-		(property "Footprint" "Capacitor_SMD:C_0402_1005Metric"
+		(property "Footprint" "proj:C_0402_1005Metric"
 			(at 317.5 53.34 0)
 			(effects
@@
 			)
 		)
-		(property "Footprint" "Capacitor_SMD:C_0402_1005Metric"
+		(property "Footprint" "proj:C_0402_1005Metric"
 			(at 317.5 63.5 0)
 			(effects
@@
 			)
 		)
-		(property "Footprint" "Resistor_SMD:R_0402_1005Metric"
+		(property "Footprint" "proj:R_0402_1005Metric"
 			(at 383.54 54.61 0)
 			(effects
@@
 			)
 		)
-		(property "Datasheet" " ~"
+		(property "Datasheet" "~"
 			(at 226.695 99.06 0)
 			(effects
@@
 			)
 		)
-		(property "Footprint" "MountingHole:MountingHole_3.2mm_M3_Pad_TopBottom"
+		(property "Footprint" "proj:standoff"
 			(at 113.03 74.93 0)
 			(effects
@@
 		(lib_id "LED:SK6812")
 		(at 180.34 153.67 0)
+		(mirror y)
 		(unit 1)
 		(exclude_from_sim no)
@@
 		(dnp no)
 		(property "Reference" "LED28"
-			(at 177.292 147.32 0)
+			(at 183.388 147.32 0)
 			(effects
 				(font
@@
 		)
 		(property "Value" "SK6812"
-			(at 190.5 149.7898 0)
+			(at 170.18 149.7898 0)
 			(effects
 				(font
@@
 		)
 		(property "Footprint" "c8:LED_SK6812_PLCC4_5.0x5.0mm_P3.2mm edit"
-			(at 181.61 161.29 0)
+			(at 179.07 161.29 0)
 			(effects
 				(font
@@
 		)
 		(property "Datasheet" "https://cdn-shop.adafruit.com/product-files/1138/SK6812+LED+datasheet+.pdf"
-			(at 182.88 163.195 0)
+			(at 177.8 163.195 0)
 			(effects
 				(font
@@
 			)
 		)
-		(property "Footprint" "Resistor_SMD:R_0402_1005Metric"
+		(property "Footprint" "proj:R_0402_1005Metric"
 			(at 347.98 128.27 0)
 			(effects
@@
 			)
 		)
-		(property "Footprint" "Capacitor_SMD:C_0402_1005Metric"
+		(property "Footprint" "proj:C_0402_1005Metric"
 			(at 345.44 64.77 0)
 			(effects
@@
 			)
 		)
-		(property "Footprint" "Resistor_SMD:R_0402_1005Metric"
+		(property "Footprint" "proj:R_0402_1005Metric"
 			(at 386.08 54.61 0)
 			(effects
@@
 			)
 		)
-		(property "Footprint" "Resistor_SMD:R_0402_1005Metric"
+		(property "Footprint" "proj:R_0402_1005Metric"
 			(at 367.03 92.71 0)
 			(effects
@@
 			)
 		)
-		(property "Footprint" "Resistor_SMD:R_0402_1005Metric"
+		(property "Footprint" "proj:R_0402_1005Metric"
 			(at 349.25 102.87 0)
 			(effects
@@
 		(lib_id "LED:SK6812")
 		(at 134.62 153.67 0)
+		(mirror y)
 		(unit 1)
 		(exclude_from_sim no)
@@
 		(dnp no)
 		(property "Reference" "LED26"
-			(at 131.572 147.32 0)
+			(at 137.668 147.32 0)
 			(effects
 				(font
@@
 		)
 		(property "Value" "SK6812"
-			(at 144.78 149.7898 0)
+			(at 124.46 149.7898 0)
 			(effects
 				(font
@@
 		)
 		(property "Footprint" "c8:LED_SK6812_PLCC4_5.0x5.0mm_P3.2mm edit"
-			(at 135.89 161.29 0)
+			(at 133.35 161.29 0)
 			(effects
 				(font
@@
 		)
 		(property "Datasheet" "https://cdn-shop.adafruit.com/product-files/1138/SK6812+LED+datasheet+.pdf"
-			(at 137.16 163.195 0)
+			(at 132.08 163.195 0)
 			(effects
 				(font

Commit message: begin matrix signaling
Parts:
- added J1: ZX-SH1.0-6PWT, Connector_JST:JST_SH_SM06B-SRSS-TB_1x06-1MP_P1.00mm_Horizontal, symbol Connector_Generic_MountingPin:Conn_01x06_MountingPin
Connections:
- net +5V: now also J1.3 (Pin_3)
- net +BATT: now also J1.1 (Pin_1)
- net +VSW: now also J1.2 (Pin_2)
- net GND: now also J1.6 (Pin_6), J1.MP (MountPin)
- net UG_HV: now also LED38.3 (DIN)
- net USB-D+: now also J1.5 (Pin_5)
- net USB-D-: now also J1.4 (Pin_4)
- net io: now reaches U12.10 (AIN5/P0.29)
- net io: now also U12.11 (AIN6/P0.30), U12.12 (AIN7/P0.31), U12.15 (AIN0/P0.02), U12.19 (AIN1/P0.03), U12.20 (AIN2/P0.04), U12.22 (P0.06), U12.24 (P0.08), U12.25 (NFC1/P0.09), U12.26 (NFC2/P0.10), U12.27 (TRACEDATA2/P0.11), U12.28 (TRACEDATA1/P0.12), U12.31 (P0.13), U12.32 (P0.14), U12.33 (P0.15), U12.34 (P0.16), U12.35 (P0.17), U12.36 (P0.21), U12.37 (P0.19), U12.38 (P0.20), U12.41 (P0.23), U12.42 (P0.24), U12.48 (P1.05), U12.49 (P1.06), U12.50 (P1.07), U12.51 (P1.08), U12.52 (TRACEDATA3/P1.09), U12.53 (P1.10), U12.54 (P1.11), U12.57 (P1.01), U12.58 (P1.02), U12.59 (P1.03), U12.6 (P0.25), U12.60 (P1.04), U12.61 (P1.12), U12.62 (P1.13), U12.63 (P1.14), U12.64 (P1.15), U12.7 (P0.26), U12.8 (P0.27), U12.9 (AIN4/P0.28)
